File: piezo-buffer-and-preamp-ritter/piezo-buffer-and-preamp-ritter_V0-2-thru.sch (EAGLE design)
At the start: 14 parts, among them Q1 MMBT2222A, Q2 548, Q3 2N5087

Commit message: new version of ritter board
Parts:
- C1: device SparkFun-Capacitors:CAP_POLPTH2 -> SparkFun-Capacitors:CAP_POLPTH4
- Q2: value 548 -> 2N5486; device CMU-ArtFab:548 -> transistor-fet:2N5486
- renumbered JP1 to MIC-SWITCH, MIC-OUT to TO-PHONE
Changed lines of the file:
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@@
 <grid distance="0.1" unitdist="inch" unit="inch" style="lines" multiple="1" display="no" altdistance="0.01" altunitdist="inch" altunit="inch"/>
 <layers>
-<layer number="1" name="Top" color="4" fill="1" visible="yes" active="no"/>
-<layer number="16" name="Bottom" color="1" fill="1" visible="yes" active="no"/>
-<layer number="17" name="Pads" color="2" fill="1" visible="yes" active="no"/>
-<layer number="18" name="Vias" color="2" fill="1" visible="yes" active="no"/>
-<layer number="19" name="Unrouted" color="6" fill="1" visible="yes" active="no"/>
-<layer number="20" name="Dimension" color="15" fill="1" visible="yes" active="no"/>
-<layer number="21" name="tPlace" color="7" fill="1" visible="yes" active="no"/>
-<layer number="22" name="bPlace" color="7" fill="1" visible="yes" active="no"/>
-<layer number="23" name="tOrigins" color="15" fill="1" visible="yes" active="no"/>
-<layer number="24" name="bOrigins" color="15" fill="1" visible="yes" active="no"/>
-<layer number="25" name="tNames" color="7" fill="1" visible="yes" active="no"/>
-<layer number="26" name="bNames" color="7" fill="1" visible="yes" active="no"/>
-<layer number="27" name="tValues" color="7" fill="1" visible="yes" active="no"/>
-<layer number="28" name="bValues" color="7" fill="1" visible="yes" active="no"/>
+<layer number="1" name="Top" color="4" fill="1" visible="no" active="no"/>
+<layer number="16" name="Bottom" color="1" fill="1" visible="no" active="no"/>
+<layer number="17" name="Pads" color="2" fill="1" visible="no" active="no"/>
+<layer number="18" name="Vias" color="2" fill="1" visible="no" active="no"/>
+<layer number="19" name="Unrouted" color="6" fill="1" visible="no" active="no"/>
+<layer number="20" name="Dimension" color="15" fill="1" visible="no" active="no"/>
+<layer number="21" name="tPlace" color="7" fill="1" visible="no" active="no"/>
+<layer number="22" name="bPlace" color="7" fill="1" visible="no" active="no"/>
+<layer number="23" name="tOrigins" color="15" fill="1" visible="no" active="no"/>
+<layer number="24" name="bOrigins" color="15" fill="1" visible="no" active="no"/>
+<layer number="25" name="tNames" color="7" fill="1" visible="no" active="no"/>
+<layer number="26" name="bNames" color="7" fill="1" visible="no" active="no"/>
+<layer number="27" name="tValues" color="7" fill="1" visible="no" active="no"/>
+<layer number="28" name="bValues" color="7" fill="1" visible="no" active="no"/>
 <layer number="29" name="tStop" color="7" fill="3" visible="no" active="no"/>
 <layer number="30" name="bStop" color="7" fill="6" visible="no" active="no"/>
@@
 <layer number="35" name="tGlue" color="7" fill="4" visible="no" active="no"/>
 <layer number="36" name="bGlue" color="7" fill="5" visible="no" active="no"/>
-<layer number="37" name="tTest" color="7" fill="1" visible="yes" active="no"/>
-<layer number="38" name="bTest" color="7" fill="1" visible="yes" active="no"/>
+<layer number="37" name="tTest" color="7" fill="1" visible="no" active="no"/>
+<layer number="38" name="bTest" color="7" fill="1" visible="no" active="no"/>
 <layer number="39" name="tKeepout" color="4" fill="11" visible="no" active="no"/>
 <layer number="40" name="bKeepout" color="1" fill="11" visible="no" active="no"/>
@@
 <layer number="44" name="Drills" color="7" fill="1" visible="no" active="no"/>
 <layer number="45" name="Holes" color="7" fill="1" visible="no" active="no"/>
-<layer number="46" name="Milling" color="3" fill="1" visible="yes" active="no"/>
-<layer number="47" name="Measures" color="7" fill="1" visible="yes" active="no"/>
-<layer number="48" name="Document" color="7" fill="1" visible="yes" active="no"/>
-<layer number="49" name="Reference" color="7" fill="1" visible="yes" active="no"/>
-<layer number="50" name="dxf" color="7" fill="1" visible="yes" active="no"/>
-<layer number="51" name="tDocu" color="7" fill="1" visible="yes" active="no"/>
-<layer number="52" name="bDocu" color="7" fill="1" visible="yes" active="no"/>
-<layer number="53" name="tGND_GNDA" color="7" fill="9" visible="yes" active="no"/>
-<layer number="54" name="bGND_GNDA" color="1" fill="9" visible="yes" active="no"/>
-<layer number="56" name="wert" color="7" fill="1" visible="yes" active="no"/>
-<layer number="57" name="tCAD" color="7" fill="1" visible="yes" active="no"/>
-<layer number="59" name="tCarbon" color="7" fill="1" visible="yes" active="no"/>
-<layer number="60" name="bCarbon" color="7" fill="1" visible="yes" active="no"/>
+<layer number="46" name="Milling" color="3" fill="1" visible="no" active="no"/>
+<layer number="47" name="Measures" color="7" fill="1" visible="no" active="no"/>
+<layer number="48" name="Document" color="7" fill="1" visible="no" active="no"/>
+<layer number="49" name="Reference" color="7" fill="1" visible="no" active="no"/>
+<layer number="50" name="dxf" color="7" fill="1" visible="no" active="no"/>
+<layer number="51" name="tDocu" color="7" fill="1" visible="no" active="no"/>
+<layer number="52" name="bDocu" color="7" fill="1" visible="no" active="no"/>
+<layer number="53" name="tGND_GNDA" color="7" fill="9" visible="no" active="no"/>
+<layer number="54" name="bGND_GNDA" color="1" fill="9" visible="no" active="no"/>
+<layer number="56" name="wert" color="7" fill="1" visible="no" active="no"/>
+<layer number="57" name="tCAD" color="7" fill="1" visible="no" active="no"/>
+<layer number="59" name="tCarbon" color="7" fill="1" visible="no" active="no"/>
+<layer number="60" name="bCarbon" color="7" fill="1" visible="no" active="no"/>
 <layer number="90" name="Modules" color="5" fill="1" visible="yes" active="yes"/>
 <layer number="91" name="Nets" color="2" fill="1" visible="yes" active="yes"/>
@@
 <part name="P+2" library="supply1" deviceset="V+" device=""/>
 <part name="SUPPLY6" library="supply2" deviceset="GND" device=""/>
-<part name="C1" library="SparkFun-Capacitors" deviceset="CAP_POL" device="PTH2" value="1000"/>
-<part name="Q2" library="CMU-ArtFab" deviceset="?548*" device=""/>
-<part name="MIC-OUT" library="SparkFun-Connectors" deviceset="AUDIO-JACK3" device=""/>
-<part name="JP1" library="SparkFun-Connectors" deviceset="M03" device="LOCK"/>
+<part name="C1" library="SparkFun-Capacitors" deviceset="CAP_POL" device="PTH4" value="1000"/>
+<part name="TO-PHONE" library="SparkFun-Connectors" deviceset="AUDIO-JACK3" device=""/>
+<part name="MIC-SWITCH" library="SparkFun-Connectors" deviceset="M03" device="LOCK"/>
 <part name="TO-HEADSET" library="SparkFun-Connectors" deviceset="AUDIO-JACK3" device=""/>
+<part name="Q2" library="transistor-fet" deviceset="?548*" device="2N" technology="6"/>
 </parts>
 <sheets>
@@
 <instance part="SUPPLY6" gate="GND" x="93.98" y="101.6"/>
 <instance part="C1" gate="G$1" x="43.18" y="40.64"/>
-<instance part="Q2" gate="G$1" x="38.1" y="81.28"/>
-<instance part="MIC-OUT" gate="G$1" x="127" y="73.66" smashed="yes" rot="R180">
+<instance part="TO-PHONE" gate="G$1" x="127" y="73.66" smashed="yes" rot="R180">
 <attribute name="NAME" x="132.08" y="68.072" size="1.778" layer="95" rot="R180"/>
 </instance>
-<instance part="JP1" gate="G$1" x="119.38" y="53.34" rot="R180"/>
+<instance part="MIC-SWITCH" gate="G$1" x="119.38" y="53.34" rot="R180"/>
 <instance part="TO-HEADSET" gate="G$1" x="127" y="93.98" smashed="yes" rot="R180">
 <attribute name="NAME" x="132.08" y="88.392" size="1.778" layer="95" rot="R180"/>
 </instance>
+<instance part="Q2" gate="G$1" x="38.1" y="81.28"/>
 </instances>
 <busses>
@@
 <pinref part="SUPPLY5" gate="GND" pin="GND"/>
 <wire x1="99.06" y1="78.74" x2="99.06" y2="50.8" width="0.1524" layer="91"/>
-<pinref part="MIC-OUT" gate="G$1" pin="RING2"/>
+<pinref part="TO-PHONE" gate="G$1" pin="RING2"/>
 <wire x1="121.92" y1="78.74" x2="99.06" y2="78.74" width="0.1524" layer="91"/>
 <wire x1="99.06" y1="78.74" x2="99.06" y2="99.06" width="0.1524" layer="91"/>
@@
 <pinref part="Q1" gate="G$1" pin="E"/>
 <wire x1="93.98" y1="63.5" x2="93.98" y2="55.88" width="0.1524" layer="91"/>
-<pinref part="JP1" gate="G$1" pin="1"/>
+<pinref part="MIC-SWITCH" gate="G$1" pin="1"/>
 <wire x1="93.98" y1="55.88" x2="111.76" y2="55.88" width="0.1524" layer="91"/>
 </segment>
@@
 <net name="TO-PHONE" class="0">
 <segment>
-<pinref part="MIC-OUT" gate="G$1" pin="EARTH"/>
+<pinref part="TO-PHONE" gate="G$1" pin="EARTH"/>
 <wire x1="121.92" y1="68.58" x2="104.14" y2="68.58" width="0.1524" layer="91"/>
 <wire x1="104.14" y1="68.58" x2="104.14" y2="53.34" width="0.1524" layer="91"/>
-<pinref part="JP1" gate="G$1" pin="2"/>
+<pinref part="MIC-SWITCH" gate="G$1" pin="2"/>
 <wire x1="104.14" y1="53.34" x2="111.76" y2="53.34" width="0.1524" layer="91"/>
 </segment>
@@
 <wire x1="121.92" y1="88.9" x2="101.6" y2="88.9" width="0.1524" layer="91"/>
 <wire x1="101.6" y1="88.9" x2="101.6" y2="50.8" width="0.1524" layer="91"/>
-<pinref part="JP1" gate="G$1" pin="3"/>
+<pinref part="MIC-SWITCH" gate="G$1" pin="3"/>
 <wire x1="101.6" y1="50.8" x2="111.76" y2="50.8" width="0.1524" layer="91"/>
 </segment>
@@
 <net name="N$8" class="0">
 <segment>
-<pinref part="MIC-OUT" gate="G$1" pin="TIP"/>
+<pinref part="TO-PHONE" gate="G$1" pin="TIP"/>
 <wire x1="121.92" y1="76.2" x2="111.76" y2="76.2" width="0.1524" layer="91"/>
 <wire x1="111.76" y1="76.2" x2="111.76" y2="96.52" width="0.1524" layer="91"/>
@@
 <net name="N$9" class="0">
 <segment>
-<pinref part="MIC-OUT" gate="G$1" pin="RING1"/>
+<pinref part="TO-PHONE" gate="G$1" pin="RING1"/>
 <wire x1="121.92" y1="71.12" x2="106.68" y2="71.12" width="0.1524" layer="91"/>
 <wire x1="106.68" y1="71.12" x2="106.68" y2="91.44" width="0.1524" layer="91"/>
