File: piezo-buffer-and-preamp-ritter/piezo-buffer-and-preamp-ritter_V0-3-thru.sch (EAGLE design)
At the start: 14 parts, among them Q1 MMBT2222A, Q2 2N5486, Q3 2N5087

Commit message: version 3 of ritter board
Parts:
- BAT1: device SparkFun-Electromechanical:BATTERYAAA-KIT -> Daniel:BATTERYAAA-KIT
Changed lines of the file:
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@@
 <part name="TO-HEADSET" library="SparkFun-Connectors" deviceset="AUDIO-JACK3" device=""/>
 <part name="Q2" library="transistor-fet" deviceset="?548*" device="2N" technology="6"/>
-<part name="BAT1" library="SparkFun-Electromechanical" deviceset="BATTERY" device="AAA-KIT"/>
+<part name="BAT1" library="Daniel" deviceset="BATTERY" device="AAA-KIT"/>
 </parts>
 <sheets>
