File: piezo-preamp-tickler-V0/piezo-preamp-tickler_V0-8.sch (EAGLE design)
At the start: 23 parts, among them IC1 TLC272, Q4 2N5484

Commit message: tickler v8
Parts:
- R9: device adafruit:TRIMPOT3386 -> Daniel:TRIM3386
- TO-HEADSET, TO-PHONE: value AUDIO-JACK3 -> AUDIO-JACK3LGPADS; device SparkFun-Connectors:AUDIO-JACK3 -> Daniel:AUDIO-JACK3LGPADS
Changed lines of the file:
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@@
 <part name="R7" library="resistor" deviceset="R-US_" device="0204/2V" value="1K"/>
 <part name="R8" library="resistor" deviceset="R-US_" device="0204/2V" value="1K"/>
-<part name="R9" library="adafruit" deviceset="TRIMPOT" device="3386"/>
+<part name="R9" library="Daniel" deviceset="TRIM" device="3386"/>
 <part name="SUPPLY6" library="supply2" deviceset="GND" device=""/>
 <part name="R2" library="resistor" deviceset="R-US_" device="0204/2V" value="1.2K"/>
@@
 <part name="SUPPLY1" library="supply2" deviceset="GND" device=""/>
 <part name="SUPPLY2" library="supply2" deviceset="GND" device=""/>
-<part name="TO-PHONE" library="SparkFun-Connectors" deviceset="AUDIO-JACK3" device=""/>
+<part name="TO-PHONE" library="Daniel" deviceset="AUDIO-JACK3" device="LGPADS"/>
 <part name="INPUT-SELECT" library="Daniel" deviceset="M03" device="SINGLE-POLE-DOUBLE-THROW"/>
-<part name="TO-HEADSET" library="SparkFun-Connectors" deviceset="AUDIO-JACK3" device=""/>
+<part name="TO-HEADSET" library="Daniel" deviceset="AUDIO-JACK3" device="LGPADS"/>
 <part name="ON/OFF" library="Daniel" deviceset="M03" device="SINGLE-POLE-DOUBLE-THROW" value="labl"/>
 </parts>
@@
 <segment>
 <wire x1="96.52" y1="27.94" x2="91.44" y2="27.94" width="0.1524" layer="91"/>
-<wire x1="76.2" y1="12.7" x2="76.2" y2="17.78" width="0.1524" layer="91"/>
+<wire x1="71.12" y1="17.78" x2="76.2" y2="17.78" width="0.1524" layer="91"/>
 <wire x1="76.2" y1="17.78" x2="96.52" y2="17.78" width="0.1524" layer="91"/>
 <wire x1="96.52" y1="17.78" x2="96.52" y2="27.94" width="0.1524" layer="91"/>
@@
 <pinref part="IC1" gate="B" pin="OUT"/>
 <pinref part="C1" gate="G$1" pin="+"/>
-<wire x1="76.2" y1="12.7" x2="66.04" y2="10.16" width="0.1524" layer="91"/>
 <pinref part="R9" gate="G$1" pin="S"/>
-<wire x1="76.2" y1="17.78" x2="71.12" y2="17.78" width="0.1524" layer="91"/>
 <wire x1="71.12" y1="17.78" x2="71.12" y2="15.24" width="0.1524" layer="91"/>
 <pinref part="R9" gate="G$1" pin="A"/>
+<wire x1="66.04" y1="7.62" x2="76.2" y2="7.62" width="0.1524" layer="91"/>
+<wire x1="76.2" y1="7.62" x2="76.2" y2="17.78" width="0.1524" layer="91"/>
+<junction x="76.2" y="17.78"/>
 </segment>
 </net>
@@
 <pinref part="R8" gate="G$1" pin="2"/>
 <pinref part="R9" gate="G$1" pin="E"/>
-<wire x1="71.12" y1="22.86" x2="66.04" y2="20.32" width="0.1524" layer="91"/>
-</segment>
-</net>
+<wire x1="71.12" y1="22.86" x2="66.04" y2="22.86" width="0.1524" layer="91"/>
+</segment>
+</net>
