File: piezo-preamp-tickler-V0/piezo-preamp-tickler_V0-5b.brd (EAGLE design)
At the start: 73.3 x 39.4 mm, 22 parts, among them IC1 TLC272, Q4 2N5484

Commit message: changes to piezo-preamp-tickler-V0-5
Parts:
- removed TO-HEADSET, TO-PHONE: AUDIO-JACK3, SparkFun-Connectors:AUDIO-JACK-TRRS-SMD
- added HEADSET, PHONE: (no value), CMU-ArtFab:1X04_LOCK
Connections:
- net GND: now also HEADSET.3, PHONE.3; no longer TO-HEADSET.RING2, TO-PHONE.RING2
- net N$12: now also HEADSET.4; no longer TO-HEADSET.EARTH
- net N$13: now also HEADSET.1, PHONE.1; no longer TO-HEADSET.TIP, TO-PHONE.TIP
- net N$15: now also HEADSET.2, PHONE.2; no longer TO-HEADSET.RING1, TO-PHONE.RING1
- net TO-PHONE: now also PHONE.4; no longer TO-PHONE.EARTH
Routing:
- net N$12: track 16.3 -> 33.9 mm
- net N$13: track 13.4 -> 8.89 mm
- net N$15: track 11.9 -> 8.89 mm
- net TO-PHONE: track 12.3 -> 14.4 mm
Changed lines of the file:
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@@
 <element name="R10" library="resistor" package="0204V" value="1K" x="16.51" y="22.225" rot="R270"/>
 <element name="BAT1" library="Daniel" package="BATTERY-A23" value="" x="66.04" y="19.685" rot="R270"/>
-<element name="TO-PHONE" library="SparkFun-Connectors" package="AUDIO-JACK-TRRS-SMD" value="AUDIO-JACK3" x="16.51" y="0" rot="MR90"/>
 <element name="INPUT-SELECT" library="SparkFun-Connectors" package="1X03_LOCK" value="" x="4.445" y="10.795"/>
-<element name="TO-HEADSET" library="SparkFun-Connectors" package="AUDIO-JACK-TRRS-SMD" value="AUDIO-JACK3" x="26.67" y="0" rot="MR90"/>
+<element name="HEADSET" library="CMU-ArtFab" package="1X04_LOCK" value="" x="26.67" y="12.7" rot="R270"/>
+<element name="PHONE" library="CMU-ArtFab" package="1X04_LOCK" value="" x="17.78" y="12.7" rot="R270"/>
 </elements>
 <signals>
@@
 <contactref element="D2" pad="C"/>
 <contactref element="R3" pad="1"/>
-<contactref element="TO-PHONE" pad="RING2"/>
-<contactref element="TO-HEADSET" pad="RING2"/>
+<contactref element="HEADSET" pad="3"/>
+<contactref element="PHONE" pad="3"/>
 </signal>
 <signal name="N$1">
@@
 <wire x1="52.75" y1="37.25" x2="44.5" y2="29" width="0.8128" layer="16"/>
 <wire x1="44.5" y1="21.75" x2="44.45" y2="21.59" width="0.6" layer="16"/>
-<wire x1="32.5" y1="4.746" x2="34" y2="6.5" width="0.8128" layer="16"/>
-<wire x1="16" y1="4.746" x2="32.5" y2="4.746" width="0.8128" layer="16"/>
 <wire x1="6.25" y1="35.905" x2="1.365" y2="29.75" width="0.8128" layer="16"/>
 <wire x1="39.25" y1="35.905" x2="6.25" y2="35.905" width="0.8128" layer="16"/>
@@
 <wire x1="1.365" y1="29.75" x2="1.365" y2="3.715" width="0.8128" layer="16"/>
 <wire x1="1.365" y1="3.715" x2="3.81" y2="1.905" width="0.8128" layer="16"/>
-<wire x1="3.81" y1="1.905" x2="12.905" y2="1.905" width="0.8128" layer="16"/>
-<wire x1="12.905" y1="1.905" x2="16" y2="4.746" width="0.8128" layer="16"/>
+<wire x1="3.81" y1="1.905" x2="28.575" y2="1.905" width="0.8128" layer="16"/>
+<wire x1="28.575" y1="1.905" x2="33.02" y2="6.35" width="0.8128" layer="16"/>
+<wire x1="33.02" y1="6.35" x2="34.29" y2="6.35" width="0.8128" layer="16"/>
 </signal>
 <signal name="N$5">
@@
 </signal>
 <signal name="TO-PHONE">
-<contactref element="TO-PHONE" pad="EARTH"/>
 <contactref element="INPUT-SELECT" pad="2"/>
+<contactref element="PHONE" pad="4"/>
 <wire x1="6.985" y1="10.668" x2="6.985" y2="8.255" width="0.8128" layer="16"/>
-<wire x1="6.985" y1="8.255" x2="7.62" y2="7.62" width="0.8128" layer="16"/>
-<wire x1="7.62" y1="7.62" x2="12.7" y2="7.62" width="0.8128" layer="16"/>
-<wire x1="12.7" y1="7.62" x2="12.7" y2="10.74" width="0.8128" layer="16"/>
-<wire x1="12.7" y1="10.74" x2="13.26" y2="11.3" width="0.6" layer="16"/>
+<wire x1="6.985" y1="8.255" x2="10.16" y2="5.08" width="0.8128" layer="16"/>
+<wire x1="10.16" y1="5.08" x2="17.653" y2="5.08" width="0.8128" layer="16"/>
 </signal>
 <signal name="N$12">
-<contactref element="TO-HEADSET" pad="EARTH"/>
 <contactref element="INPUT-SELECT" pad="3"/>
 <wire x1="9.525" y1="10.922" x2="12.573" y2="13.97" width="0.8128" layer="16"/>
-<wire x1="12.573" y1="13.97" x2="20.32" y2="13.97" width="0.8128" layer="16"/>
-<wire x1="20.32" y1="13.97" x2="22.99" y2="11.3" width="0.8128" layer="16"/>
-<wire x1="22.99" y1="11.3" x2="23.42" y2="11.3" width="0.8128" layer="16"/>
+<contactref element="HEADSET" pad="4"/>
+<wire x1="12.573" y1="13.97" x2="12.7" y2="13.97" width="0.8128" layer="16"/>
+<wire x1="12.7" y1="13.97" x2="13.97" y2="15.24" width="0.8128" layer="16"/>
+<wire x1="13.97" y1="15.24" x2="27.94" y2="15.24" width="0.8128" layer="16"/>
+<wire x1="27.94" y1="15.24" x2="30.48" y2="12.7" width="0.8128" layer="16"/>
+<wire x1="30.48" y1="12.7" x2="30.48" y2="7.62" width="0.8128" layer="16"/>
+<wire x1="30.48" y1="7.62" x2="27.94" y2="5.08" width="0.8128" layer="16"/>
+<wire x1="27.94" y1="5.08" x2="26.543" y2="5.08" width="0.8128" layer="16"/>
 </signal>
 <signal name="N$13">
-<contactref element="TO-PHONE" pad="TIP"/>
-<contactref element="TO-HEADSET" pad="TIP"/>
-<wire x1="24.75" y1="8.73" x2="20" y2="8.73" width="0.8128" layer="16"/>
-<wire x1="26" y1="11.25" x2="24.75" y2="8.73" width="0.8128" layer="16"/>
-<wire x1="27.75" y1="11.25" x2="26" y2="11.25" width="0.8128" layer="16"/>
-<wire x1="28.75" y1="10.25" x2="27.75" y2="11.25" width="0.8128" layer="16"/>
-<wire x1="29.75" y1="10.25" x2="28.75" y2="10.25" width="0.6" layer="16"/>
-<wire x1="20" y1="8.73" x2="19.76" y2="10.2" width="0.6" layer="16"/>
-<wire x1="29.75" y1="10.25" x2="29.92" y2="10.2" width="0.8128" layer="16"/>
+<contactref element="HEADSET" pad="1"/>
+<contactref element="PHONE" pad="1"/>
+<wire x1="17.907" y1="12.7" x2="26.797" y2="12.7" width="0.8128" layer="16"/>
 </signal>
 <signal name="N$15">
-<contactref element="TO-PHONE" pad="RING1"/>
-<contactref element="TO-HEADSET" pad="RING1"/>
-<wire x1="29.75" y1="7.27" x2="20" y2="7.27" width="0.8128" layer="16"/>
-<wire x1="20" y1="7.27" x2="19.76" y2="6.2" width="0.6" layer="16"/>
-<wire x1="29.75" y1="7.27" x2="29.92" y2="6.2" width="0.6" layer="16"/>
+<contactref element="HEADSET" pad="2"/>
+<contactref element="PHONE" pad="2"/>
+<wire x1="17.653" y1="10.16" x2="26.543" y2="10.16" width="0.8128" layer="16"/>
 </signal>
 </signals>
