File: piezo-preamp-tickler-V0/piezo-preamp-tickler_V2-RevA.sch (EAGLE design)
At the start: 37 parts, among them IC1 OPA2134UA, IC2 SST5484, Q1 SST201

Commit message: new tickler board
Parts:
- added SW1: (no value), microbuilder:SWITCH_DPDT
- R1: value 100K -> 2.2K
Connections:
- new net N$26: SW1.O1, TO-PHONE.RING1
- new net N$27: SW1.O2, TO-PHONE.TIP
- net N$11: now also SW1.S1, SW1.S2
- net N$13: now also SW1.P2; no longer TO-PHONE.TIP
- net N$15: now also SW1.P1; no longer TO-PHONE.RING1
Other:
- moved on the sheet: R10, TO-HEADSET
Changed lines of the file:
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@@
 <part name="R8" library="CMU-ArtFab" deviceset="R-US_" device="R0603" value="500"/>
 <part name="R2" library="CMU-ArtFab" deviceset="R-US_" device="R0603" value="1.2K"/>
-<part name="R1" library="CMU-ArtFab" deviceset="R-US_" device="R0603" value="100K"/>
+<part name="R1" library="CMU-ArtFab" deviceset="R-US_" device="R0603" value="2.2K"/>
 <part name="R3" library="CMU-ArtFab" deviceset="R-US_" device="R0603" value="1M"/>
 <part name="R10" library="CMU-ArtFab" deviceset="R-US_" device="R0603" value="1K"/>
@@
 <attribute name="DIGIKEY" value="399-8282-1-ND"/>
 </part>
+<part name="SW1" library="microbuilder" deviceset="SWITCH_DPDT" device="">
+<attribute name="BOTTOM" value="buffer2-phone"/>
+<attribute name="DIGIKEY" value="401-2002-1-ND"/>
+<attribute name="DIGIKEY2" value="563-1342-1-ND"/>
+<attribute name="TOP" value="opamp"/>
+</part>
 </parts>
 <sheets>
@@
 <instance part="R1" gate="G$1" x="165.1" y="27.94" rot="R90"/>
 <instance part="R3" gate="G$1" x="129.54" y="27.94" rot="R90"/>
-<instance part="R10" gate="G$1" x="119.38" y="38.1" rot="R180"/>
+<instance part="R10" gate="G$1" x="121.92" y="38.1" rot="R180"/>
 <instance part="SUPPLY1" gate="GND" x="129.54" y="12.7"/>
-<instance part="SUPPLY2" gate="GND" x="175.26" y="45.72"/>
+<instance part="SUPPLY2" gate="GND" x="175.26" y="12.7"/>
 <instance part="TO-PHONE" gate="G$1" x="220.98" y="58.42" smashed="yes" rot="R180">
 <attribute name="NAME" x="226.06" y="52.832" size="1.778" layer="95" rot="R180"/>
 </instance>
-<instance part="TO-HEADSET" gate="G$1" x="203.2" y="78.74" smashed="yes" rot="R180">
-<attribute name="NAME" x="208.28" y="73.152" size="1.778" layer="95" rot="R180"/>
+<instance part="TO-HEADSET" gate="G$1" x="220.98" y="78.74" smashed="yes" rot="R180">
+<attribute name="NAME" x="226.06" y="73.152" size="1.778" layer="95" rot="R180"/>
 </instance>
 <instance part="IC1" gate="A" x="43.18" y="30.48" smashed="yes">
@@
 <attribute name="DIGIKEY" x="-22.098" y="24.13" size="0.6096" layer="96" display="both"/>
 </instance>
+<instance part="SW1" gate="G$1" x="152.4" y="78.74" rot="R180">
+<attribute name="BOTTOM" x="151.13" y="82.55" size="0.6096" layer="96" rot="R180" display="both"/>
+<attribute name="TOP" x="151.384" y="87.63" size="0.6096" layer="96" rot="R180" display="both"/>
+<attribute name="DIGIKEY" x="165.1" y="79.502" size="0.6096" layer="96" rot="R180" display="both"/>
+<attribute name="DIGIKEY2" x="165.608" y="78.232" size="0.6096" layer="96" rot="R180" display="both"/>
+</instance>
 </instances>
 <busses>
@@
 <segment>
 <pinref part="SUPPLY2" gate="GND" pin="GND"/>
-<wire x1="175.26" y1="63.5" x2="175.26" y2="48.26" width="0.1524" layer="91"/>
+<wire x1="175.26" y1="63.5" x2="175.26" y2="15.24" width="0.1524" layer="91"/>
 <pinref part="TO-PHONE" gate="G$1" pin="RING2"/>
 <wire x1="215.9" y1="63.5" x2="175.26" y2="63.5" width="0.1524" layer="91"/>
@@
 <junction x="175.26" y="63.5"/>
 <pinref part="TO-HEADSET" gate="G$1" pin="RING2"/>
-<wire x1="175.26" y1="83.82" x2="198.12" y2="83.82" width="0.1524" layer="91"/>
+<wire x1="175.26" y1="83.82" x2="215.9" y2="83.82" width="0.1524" layer="91"/>
 </segment>
 <segment>
@@
 <wire x1="129.54" y1="33.02" x2="129.54" y2="38.1" width="0.1524" layer="91"/>
 <pinref part="R10" gate="G$1" pin="1"/>
-<wire x1="124.46" y1="38.1" x2="129.54" y2="38.1" width="0.1524" layer="91"/>
+<wire x1="127" y1="38.1" x2="129.54" y2="38.1" width="0.1524" layer="91"/>
 <junction x="129.54" y="38.1"/>
 <pinref part="D1" gate="G$1" pin="C"/>
@@
 <wire x1="111.76" y1="38.1" x2="114.3" y2="38.1" width="0.1524" layer="91"/>
 <pinref part="C1" gate="G$1" pin="2"/>
+<pinref part="SW1" gate="G$1" pin="S2"/>
+<wire x1="114.3" y1="38.1" x2="116.84" y2="38.1" width="0.1524" layer="91"/>
+<wire x1="149.86" y1="86.36" x2="114.3" y2="86.36" width="0.1524" layer="91"/>
+<wire x1="114.3" y1="86.36" x2="114.3" y2="76.2" width="0.1524" layer="91"/>
+<junction x="114.3" y="38.1"/>
+<pinref part="SW1" gate="G$1" pin="S1"/>
+<wire x1="114.3" y1="76.2" x2="114.3" y2="38.1" width="0.1524" layer="91"/>
+<wire x1="149.86" y1="76.2" x2="114.3" y2="76.2" width="0.1524" layer="91"/>
+<junction x="114.3" y="76.2"/>
 </segment>
 </net>
@@
 <segment>
 <pinref part="TO-HEADSET" gate="G$1" pin="EARTH"/>
-<wire x1="198.12" y1="73.66" x2="177.8" y2="73.66" width="0.1524" layer="91"/>
+<wire x1="215.9" y1="73.66" x2="177.8" y2="73.66" width="0.1524" layer="91"/>
 <wire x1="177.8" y1="73.66" x2="177.8" y2="48.26" width="0.1524" layer="91"/>
 <wire x1="177.8" y1="48.26" x2="190.5" y2="48.26" width="0.1524" layer="91"/>
@@
 <net name="N$13" class="0">
 <segment>
-<pinref part="TO-PHONE" gate="G$1" pin="TIP"/>
-<wire x1="215.9" y1="60.96" x2="187.96" y2="60.96" width="0.1524" layer="91"/>
-<wire x1="187.96" y1="60.96" x2="187.96" y2="81.28" width="0.1524" layer="91"/>
 <pinref part="TO-HEADSET" gate="G$1" pin="TIP"/>
-<wire x1="187.96" y1="81.28" x2="198.12" y2="81.28" width="0.1524" layer="91"/>
+<wire x1="215.9" y1="81.28" x2="160.02" y2="81.28" width="0.1524" layer="91"/>
+<pinref part="SW1" gate="G$1" pin="P2"/>
+<wire x1="160.02" y1="81.28" x2="160.02" y2="83.82" width="0.1524" layer="91"/>
+<wire x1="160.02" y1="83.82" x2="157.48" y2="83.82" width="0.1524" layer="91"/>
 </segment>
 </net>
 <net name="N$15" class="0">
 <segment>
-<pinref part="TO-PHONE" gate="G$1" pin="RING1"/>
-<wire x1="215.9" y1="55.88" x2="182.88" y2="55.88" width="0.1524" layer="91"/>
-<wire x1="182.88" y1="55.88" x2="182.88" y2="76.2" width="0.1524" layer="91"/>
 <pinref part="TO-HEADSET" gate="G$1" pin="RING1"/>
-<wire x1="182.88" y1="76.2" x2="198.12" y2="76.2" width="0.1524" layer="91"/>
+<wire x1="160.02" y1="76.2" x2="215.9" y2="76.2" width="0.1524" layer="91"/>
+<pinref part="SW1" gate="G$1" pin="P1"/>
+<wire x1="160.02" y1="76.2" x2="160.02" y2="73.66" width="0.1524" layer="91"/>
+<wire x1="160.02" y1="73.66" x2="157.48" y2="73.66" width="0.1524" layer="91"/>
 </segment>
 </net>
@@
 </segment>
 </net>
+<net name="N$26" class="0">
+<segment>
+<pinref part="TO-PHONE" gate="G$1" pin="RING1"/>
+<wire x1="215.9" y1="55.88" x2="144.78" y2="55.88" width="0.1524" layer="91"/>
+<wire x1="144.78" y1="55.88" x2="144.78" y2="71.12" width="0.1524" layer="91"/>
+<pinref part="SW1" gate="G$1" pin="O1"/>
+<wire x1="144.78" y1="71.12" x2="149.86" y2="71.12" width="0.1524" layer="91"/>
+</segment>
+</net>
+<net name="N$27" class="0">
+<segment>
+<pinref part="TO-PHONE" gate="G$1" pin="TIP"/>
+<wire x1="215.9" y1="60.96" x2="139.7" y2="60.96" width="0.1524" layer="91"/>
+<wire x1="139.7" y1="60.96" x2="139.7" y2="81.28" width="0.1524" layer="91"/>
+<pinref part="SW1" gate="G$1" pin="O2"/>
+<wire x1="139.7" y1="81.28" x2="149.86" y2="81.28" width="0.1524" layer="91"/>
+</segment>
+</net>

Commit message: new tickler board
Parts:
- SW1-DPDT: value (none) -> OUTPUT-select
- SW2-SPST: value SPDT -> INPUT-select
- renumbered MIC-SELECT to SW2-SPST, SW1 to SW1-DPDT
Other:
- note added: "Buffer-Stage-1"
- note added: "Buffer-Stage-2"
- note added: "OpAmp-Amplifier"
Changed lines of the file:
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@@
 <part name="D1" library="diode" deviceset="DIODE-" device="SOD123"/>
 <part name="D2" library="diode" deviceset="DIODE-" device="SOD123"/>
-<part name="MIC-SELECT" library="CMU-ArtFab" deviceset="SWITCH_SPDT" device="TE-CONNECT" value="SPDT"/>
+<part name="SW2-SPST" library="CMU-ArtFab" deviceset="SWITCH_SPDT" device="TE-CONNECT" value="INPUT-select"/>
 <part name="C2" library="adafruit" deviceset="C-US" device="C0805K" value="0.1uF"/>
 <part name="C1" library="adafruit" deviceset="C-US" device="C0805K" value="10uF"/>
@@
 <attribute name="DIGIKEY" value="399-8282-1-ND"/>
 </part>
-<part name="SW1" library="microbuilder" deviceset="SWITCH_DPDT" device="">
+<part name="SW1-DPDT" library="microbuilder" deviceset="SWITCH_DPDT" device="" value="OUTPUT-select">
 <attribute name="BOTTOM" value="buffer2-phone"/>
 <attribute name="DIGIKEY" value="401-2002-1-ND"/>
@@
 <sheet>
 <plain>
+<text x="-91.44" y="78.74" size="1.778" layer="91">Buffer-Stage-1</text>
+<text x="40.64" y="81.28" size="1.778" layer="91">OpAmp-Amplifier</text>
+<text x="137.16" y="10.16" size="1.778" layer="91">Buffer-Stage-2</text>
 </plain>
 <instances>
@@
 <instance part="D1" gate="G$1" x="137.16" y="30.48" rot="R90"/>
 <instance part="D2" gate="G$1" x="137.16" y="22.86" rot="R270"/>
-<instance part="MIC-SELECT" gate="G$1" x="195.58" y="50.8" rot="R180"/>
+<instance part="SW2-SPST" gate="G$1" x="195.58" y="50.8" smashed="yes" rot="R180">
+<attribute name="NAME" x="191.262" y="44.958" size="1.778" layer="95"/>
+<attribute name="VALUE" x="191.262" y="40.132" size="1.778" layer="96"/>
+</instance>
 <instance part="C2" gate="G$1" x="78.74" y="60.96"/>
 <instance part="C1" gate="G$1" x="106.68" y="38.1" rot="R90"/>
@@
 <attribute name="DIGIKEY" x="-22.098" y="24.13" size="0.6096" layer="96" display="both"/>
 </instance>
-<instance part="SW1" gate="G$1" x="152.4" y="78.74" rot="R180">
+<instance part="SW1-DPDT" gate="G$1" x="152.4" y="78.74" smashed="yes" rot="R180">
 <attribute name="BOTTOM" x="151.13" y="82.55" size="0.6096" layer="96" rot="R180" display="both"/>
 <attribute name="TOP" x="151.384" y="87.63" size="0.6096" layer="96" rot="R180" display="both"/>
 <attribute name="DIGIKEY" x="165.1" y="79.502" size="0.6096" layer="96" rot="R180" display="both"/>
 <attribute name="DIGIKEY2" x="165.608" y="78.232" size="0.6096" layer="96" rot="R180" display="both"/>
+<attribute name="VALUE" x="148.082" y="64.77" size="1.27" layer="96"/>
+<attribute name="NAME" x="147.955" y="67.31" size="1.27" layer="95"/>
 </instance>
 </instances>
@@
 <wire x1="111.76" y1="38.1" x2="114.3" y2="38.1" width="0.1524" layer="91"/>
 <pinref part="C1" gate="G$1" pin="2"/>
-<pinref part="SW1" gate="G$1" pin="S2"/>
+<pinref part="SW1-DPDT" gate="G$1" pin="S2"/>
 <wire x1="114.3" y1="38.1" x2="116.84" y2="38.1" width="0.1524" layer="91"/>
 <wire x1="149.86" y1="86.36" x2="114.3" y2="86.36" width="0.1524" layer="91"/>
 <wire x1="114.3" y1="86.36" x2="114.3" y2="76.2" width="0.1524" layer="91"/>
 <junction x="114.3" y="38.1"/>
-<pinref part="SW1" gate="G$1" pin="S1"/>
+<pinref part="SW1-DPDT" gate="G$1" pin="S1"/>
 <wire x1="114.3" y1="76.2" x2="114.3" y2="38.1" width="0.1524" layer="91"/>
 <wire x1="149.86" y1="76.2" x2="114.3" y2="76.2" width="0.1524" layer="91"/>
@@
 <junction x="165.1" y="53.34"/>
 <pinref part="R1" gate="G$1" pin="2"/>
-<pinref part="MIC-SELECT" gate="G$1" pin="3"/>
+<pinref part="SW2-SPST" gate="G$1" pin="3"/>
 </segment>
 </net>
@@
 <wire x1="177.8" y1="73.66" x2="177.8" y2="48.26" width="0.1524" layer="91"/>
 <wire x1="177.8" y1="48.26" x2="190.5" y2="48.26" width="0.1524" layer="91"/>
-<pinref part="MIC-SELECT" gate="G$1" pin="1"/>
+<pinref part="SW2-SPST" gate="G$1" pin="1"/>
 </segment>
 </net>
@@
 <pinref part="TO-HEADSET" gate="G$1" pin="TIP"/>
 <wire x1="215.9" y1="81.28" x2="160.02" y2="81.28" width="0.1524" layer="91"/>
-<pinref part="SW1" gate="G$1" pin="P2"/>
+<pinref part="SW1-DPDT" gate="G$1" pin="P2"/>
 <wire x1="160.02" y1="81.28" x2="160.02" y2="83.82" width="0.1524" layer="91"/>
 <wire x1="160.02" y1="83.82" x2="157.48" y2="83.82" width="0.1524" layer="91"/>
@@
 <pinref part="TO-HEADSET" gate="G$1" pin="RING1"/>
 <wire x1="160.02" y1="76.2" x2="215.9" y2="76.2" width="0.1524" layer="91"/>
-<pinref part="SW1" gate="G$1" pin="P1"/>
+<pinref part="SW1-DPDT" gate="G$1" pin="P1"/>
 <wire x1="160.02" y1="76.2" x2="160.02" y2="73.66" width="0.1524" layer="91"/>
 <wire x1="160.02" y1="73.66" x2="157.48" y2="73.66" width="0.1524" layer="91"/>
@@
 <wire x1="208.28" y1="53.34" x2="208.28" y2="50.8" width="0.1524" layer="91"/>
 <wire x1="208.28" y1="50.8" x2="200.66" y2="50.8" width="0.1524" layer="91"/>
-<pinref part="MIC-SELECT" gate="G$1" pin="2"/>
+<pinref part="SW2-SPST" gate="G$1" pin="2"/>
 </segment>
 </net>
@@
 <wire x1="215.9" y1="55.88" x2="144.78" y2="55.88" width="0.1524" layer="91"/>
 <wire x1="144.78" y1="55.88" x2="144.78" y2="71.12" width="0.1524" layer="91"/>
-<pinref part="SW1" gate="G$1" pin="O1"/>
+<pinref part="SW1-DPDT" gate="G$1" pin="O1"/>
 <wire x1="144.78" y1="71.12" x2="149.86" y2="71.12" width="0.1524" layer="91"/>
 </segment>
@@
 <wire x1="215.9" y1="60.96" x2="139.7" y2="60.96" width="0.1524" layer="91"/>
 <wire x1="139.7" y1="60.96" x2="139.7" y2="81.28" width="0.1524" layer="91"/>
-<pinref part="SW1" gate="G$1" pin="O2"/>
+<pinref part="SW1-DPDT" gate="G$1" pin="O2"/>
 <wire x1="139.7" y1="81.28" x2="149.86" y2="81.28" width="0.1524" layer="91"/>
 </segment>
