File: piezo-preamp-tickler-V0/piezo-preamp-tickler_V2-RevB.sch (EAGLE design)
At the start: 38 parts, among them IC1 OPA2134UA, IC2 SST5484, Q1 SST201, SW1-DPDT OUTPUT-select, SW2-SPST INPUT-select

Commit message: piezo rev c
Other:
- moved on the sheet: R16
Changed lines of the file:
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@@
 <wire x1="10.16" y1="2.54" x2="-96.52" y2="2.54" width="0.1524" layer="98"/>
 <wire x1="-96.52" y1="2.54" x2="-96.52" y2="88.9" width="0.1524" layer="98"/>
-<wire x1="17.78" y1="88.9" x2="109.22" y2="88.9" width="0.1524" layer="98"/>
+<wire x1="15.24" y1="88.9" x2="109.22" y2="88.9" width="0.1524" layer="98"/>
 <wire x1="109.22" y1="88.9" x2="109.22" y2="2.54" width="0.1524" layer="98"/>
-<wire x1="109.22" y1="2.54" x2="17.78" y2="2.54" width="0.1524" layer="98"/>
-<wire x1="17.78" y1="2.54" x2="17.78" y2="88.9" width="0.1524" layer="98"/>
+<wire x1="109.22" y1="2.54" x2="15.24" y2="2.54" width="0.1524" layer="98"/>
+<wire x1="15.24" y1="2.54" x2="15.24" y2="88.9" width="0.1524" layer="98"/>
 <wire x1="111.76" y1="-2.54" x2="111.76" y2="58.42" width="0.1524" layer="98"/>
 <wire x1="111.76" y1="58.42" x2="172.72" y2="58.42" width="0.1524" layer="98"/>
@@
 <attribute name="VALUE" x="71.12" y="45.72" size="1.778" layer="96" ratio="12"/>
 </instance>
-<instance part="GND4" gate="1" x="38.1" y="7.62" smashed="yes">
-<attribute name="VALUE" x="35.56" y="5.08" size="1.778" layer="96" ratio="12"/>
+<instance part="GND4" gate="1" x="38.1" y="12.7" smashed="yes">
+<attribute name="VALUE" x="35.56" y="10.16" size="1.778" layer="96" ratio="12"/>
 </instance>
 <instance part="R5" gate="G$1" x="48.26" y="58.42" rot="R90"/>
@@
 <attribute name="NAME" x="147.955" y="67.31" size="1.27" layer="95"/>
 </instance>
-<instance part="R16" gate="G$1" x="30.48" y="15.24"/>
+<instance part="R16" gate="G$1" x="30.48" y="17.78"/>
 </instances>
 <busses>
@@
 <segment>
 <pinref part="GND4" gate="1" pin="GND"/>
-<wire x1="38.1" y1="10.16" x2="38.1" y2="22.86" width="0.1524" layer="91"/>
+<wire x1="38.1" y1="15.24" x2="38.1" y2="22.86" width="0.1524" layer="91"/>
 <pinref part="IC1" gate="A" pin="V-"/>
 </segment>
@@
 <segment>
 <wire x1="45.72" y1="30.48" x2="58.42" y2="30.48" width="0.1524" layer="91"/>
+<wire x1="58.42" y1="30.48" x2="58.42" y2="17.78" width="0.1524" layer="91"/>
 <wire x1="58.42" y1="35.56" x2="58.42" y2="30.48" width="0.1524" layer="91"/>
+<junction x="58.42" y="30.48"/>
 <pinref part="R8" gate="G$1" pin="1"/>
 <pinref part="IC1" gate="A" pin="OUT"/>
 <pinref part="R16" gate="G$1" pin="S"/>
-<wire x1="35.56" y1="15.24" x2="58.42" y2="15.24" width="0.1524" layer="91"/>
-<wire x1="58.42" y1="15.24" x2="58.42" y2="30.48" width="0.1524" layer="91"/>
-<junction x="58.42" y="30.48"/>
+<wire x1="35.56" y1="17.78" x2="58.42" y2="17.78" width="0.1524" layer="91"/>
 </segment>
 </net>
@@
 <pinref part="R9" gate="G$1" pin="E"/>
 <wire x1="68.58" y1="33.02" x2="68.58" y2="30.48" width="0.1524" layer="91"/>
-</segment>
-</net>
-<net name="N$8" class="0">
-<segment>
-<wire x1="48.26" y1="53.34" x2="25.4" y2="53.34" width="0.1524" layer="91"/>
-<wire x1="48.26" y1="53.34" x2="55.88" y2="53.34" width="0.1524" layer="91"/>
-<wire x1="55.88" y1="53.34" x2="55.88" y2="50.8" width="0.1524" layer="91"/>
-<wire x1="66.04" y1="53.34" x2="55.88" y2="53.34" width="0.1524" layer="91"/>
-<junction x="48.26" y="53.34"/>
-<junction x="55.88" y="53.34"/>
-<pinref part="R5" gate="G$1" pin="1"/>
-<pinref part="R6" gate="G$1" pin="2"/>
-<pinref part="R7" gate="G$1" pin="2"/>
-<pinref part="C3" gate="G$1" pin="1"/>
-<wire x1="25.4" y1="53.34" x2="25.4" y2="33.02" width="0.1524" layer="91"/>
-<pinref part="IC1" gate="A" pin="+IN"/>
-<wire x1="25.4" y1="33.02" x2="30.48" y2="33.02" width="0.1524" layer="91"/>
 </segment>
 </net>
@@
 </segment>
 </net>
-<net name="N$28" class="0">
+<net name="N$29" class="0">
+<segment>
+<pinref part="C3" gate="G$1" pin="1"/>
+<wire x1="55.88" y1="53.34" x2="55.88" y2="50.8" width="0.1524" layer="91"/>
+<pinref part="R7" gate="G$1" pin="2"/>
+<wire x1="66.04" y1="53.34" x2="55.88" y2="53.34" width="0.1524" layer="91"/>
+<junction x="55.88" y="53.34"/>
+<wire x1="48.26" y1="53.34" x2="55.88" y2="53.34" width="0.1524" layer="91"/>
+<junction x="48.26" y="53.34"/>
+<pinref part="R5" gate="G$1" pin="1"/>
+<pinref part="R6" gate="G$1" pin="2"/>
+<pinref part="IC1" gate="A" pin="+IN"/>
+<wire x1="48.26" y1="53.34" x2="30.48" y2="53.34" width="0.1524" layer="91"/>
+<wire x1="30.48" y1="53.34" x2="30.48" y2="33.02" width="0.1524" layer="91"/>
+</segment>
+</net>
+<net name="N$8" class="0">
 <segment>
 <pinref part="IC1" gate="A" pin="-IN"/>
-<wire x1="30.48" y1="27.94" x2="30.48" y2="20.32" width="0.1524" layer="91"/>
+<wire x1="30.48" y1="27.94" x2="5.08" y2="27.94" width="0.1524" layer="91"/>
+<wire x1="5.08" y1="27.94" x2="5.08" y2="35.56" width="0.1524" layer="91"/>
+<pinref part="R15" gate="G$1" pin="2"/>
+<wire x1="5.08" y1="35.56" x2="0" y2="35.56" width="0.1524" layer="91"/>
 <pinref part="R16" gate="G$1" pin="E"/>
-<wire x1="30.48" y1="27.94" x2="7.62" y2="27.94" width="0.1524" layer="91"/>
+<wire x1="30.48" y1="22.86" x2="30.48" y2="27.94" width="0.1524" layer="91"/>
 <junction x="30.48" y="27.94"/>
-<wire x1="7.62" y1="27.94" x2="7.62" y2="35.56" width="0.1524" layer="91"/>
-<pinref part="R15" gate="G$1" pin="2"/>
-<wire x1="0" y1="35.56" x2="7.62" y2="35.56" width="0.1524" layer="91"/>
-</segment>
-</net>
+</segment>
+</net>
