File: piezo-preamp-tickler-V0/piezo-preamp-tickler_V2-RevD.sch (EAGLE design)
At the start: 39 parts, among them IC1 OPA2134UA, Q1 J201SOT-23, Q2 J201SOT-23, SW2-SPST INPUT-select

Commit message: piezo rev d
Parts:
- removed R9: 20K, adafruit:TRIMPOTTC33X
- added D4: (no value), diode:DIODE-SOD123
- added U$4: (no value), CMU-ArtFab:POT
Connections:
- net GND: now also D4.A
- net N$2: now also D4.C
- net N$6: now also U$4.WIPER; no longer R9.S
- net N$7: now also U$4.OUT; no longer R9.E
