File: piezo-preamp-tickler-V0/piezo-preamp-tickler_V2-RevF.sch (EAGLE design)
At the start: 63 parts, among them IC1 OPA2134UA, Q1 J201SOT-23, Q2 J201SOT-23, SW2-SPST INPUT-select, U1 VREG12_SOT23-5

Commit message: piezo rev F
Parts:
- removed C11: 0.1uF, SparkFun:CAP_POL3528
- added C12: 0.1uF, adafruit:C-USC0805K
- C1: device adafruit:C-US6032 -> adafruit:C-US
- C10: device SparkFun:CAP_POL3528 -> adafruit:C-USC0805K
- C8: device SparkFun:CAP_POL3528 -> SparkFun:CAP_POL1206
- R18, R19, R20, R21, R22, R23, R24, R9: device CMU-ArtFab:R-US_R0805 -> CMU-ArtFab:R-US_R0603
- U$4, U$5: device CMU-ArtFab:POT -> CMU-ArtFab:POTTHUMBPOT14MM
Connections:
- net N$33: now also C10.2; no longer C10.-
- net N$41: now also C12.1; no longer C11.+
- net N$42: now also C12.2; no longer C11.-
- net V+: now also C10.1; no longer C10.+
Changed lines of the file:
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@@
 <?xml version="1.0" encoding="utf-8"?>
 <!DOCTYPE eagle SYSTEM "eagle.dtd">
-<eagle version="8.2.1">
+<eagle version="8.3.1">
 <drawing>
 <settings>
 <setting alwaysvectorfont="no"/>
+<setting keepoldvectorfont="yes"/>
 <setting verticaltext="up"/>
 </settings>
@@
 <part name="SW2-SPST" library="CMU-ArtFab" deviceset="SWITCH_SPDT" device="CL-SB-12B" value="INPUT-select"/>
 <part name="C2" library="adafruit" deviceset="C-US" device="C0805K" value="0.1uF"/>
-<part name="C1" library="adafruit" deviceset="C-US" device="6032" value="47uF"/>
+<part name="C1" library="adafruit" deviceset="C-US" device="" value="47uF"/>
 <part name="C3" library="adafruit" deviceset="C-US" device="C0805K" value="10uF"/>
 <part name="R14" library="CMU-ArtFab" deviceset="R-US_" device="R0603" value="1.2K"/>
@@
 <part name="U$2" library="CMU-ArtFab" deviceset="SWITCH_DPDT" device=""/>
 <part name="D4" library="diode" library_urn="urn:adsk.eagle:library:210" deviceset="DIODE-" device="SOD123"/>
-<part name="U$4" library="CMU-ArtFab" deviceset="POT" device=""/>
+<part name="U$4" library="CMU-ArtFab" deviceset="POT" device="THUMBPOT14MM"/>
 <part name="C7" library="adafruit" deviceset="C-US" device="C0805K" value="3.3pF"/>
-<part name="U$5" library="CMU-ArtFab" deviceset="POT" device=""/>
+<part name="U$5" library="CMU-ArtFab" deviceset="POT" device="THUMBPOT14MM"/>
 <part name="U$6" library="microbuilder" deviceset="VBAT" device=""/>
 <part name="D7" library="SparkFun" deviceset="DIODE" device="SMA" value="10BQ015"/>
@@
 <part name="GND18" library="SparkFun" deviceset="GND" device=""/>
 <part name="U1" library="CMU-ArtFab" deviceset="VREG12_SOT23-5" device=""/>
-<part name="R9" library="CMU-ArtFab" deviceset="R-US_" device="R0805" value="866k"/>
-<part name="R18" library="CMU-ArtFab" deviceset="R-US_" device="R0805" value="100k"/>
-<part name="C8" library="SparkFun" deviceset="CAP_POL" device="3528" value="2.2pf"/>
-<part name="R19" library="CMU-ArtFab" deviceset="R-US_" device="R0805" value="15k"/>
+<part name="R9" library="CMU-ArtFab" deviceset="R-US_" device="R0603" value="866k"/>
+<part name="R18" library="CMU-ArtFab" deviceset="R-US_" device="R0603" value="100k"/>
+<part name="C8" library="SparkFun" deviceset="CAP_POL" device="1206" value="2.2pf"/>
+<part name="R19" library="CMU-ArtFab" deviceset="R-US_" device="R0603" value="15k"/>
 <part name="C9" library="SparkFun" deviceset="CAP_POL" device="3528" value="56nf"/>
 <part name="GND1" library="SparkFun" deviceset="GND" device=""/>
@@
 <part name="U$7" library="CMU-ArtFab" deviceset="DW01A" device=""/>
 <part name="U$9" library="CMU-ArtFab" deviceset="F8205A" device=""/>
-<part name="C10" library="SparkFun" deviceset="CAP_POL" device="3528" value="0.1uF"/>
-<part name="R20" library="CMU-ArtFab" deviceset="R-US_" device="R0805" value="1.2k"/>
+<part name="R20" library="CMU-ArtFab" deviceset="R-US_" device="R0603" value="1.2k"/>
 <part name="LED2" library="led" library_urn="urn:adsk.eagle:library:259" deviceset="LED" device="3MM"/>
 <part name="LED3" library="led" library_urn="urn:adsk.eagle:library:259" deviceset="LED" device="3MM"/>
 <part name="U$11" library="microbuilder" deviceset="VBAT" device=""/>
-<part name="R21" library="CMU-ArtFab" deviceset="R-US_" device="R0805" value="1k"/>
-<part name="R22" library="CMU-ArtFab" deviceset="R-US_" device="R0805" value="1k"/>
+<part name="R21" library="CMU-ArtFab" deviceset="R-US_" device="R0603" value="1k"/>
+<part name="R22" library="CMU-ArtFab" deviceset="R-US_" device="R0603" value="1k"/>
 <part name="P+1" library="supply1" library_urn="urn:adsk.eagle:library:371" deviceset="V+" device=""/>
 <part name="P+4" library="supply1" library_urn="urn:adsk.eagle:library:371" deviceset="V+" device=""/>
-<part name="C11" library="SparkFun" deviceset="CAP_POL" device="3528" value="0.1uF"/>
-<part name="R23" library="CMU-ArtFab" deviceset="R-US_" device="R0805" value="100"/>
+<part name="R23" library="CMU-ArtFab" deviceset="R-US_" device="R0603" value="100"/>
 <part name="U$12" library="microbuilder" deviceset="VBAT" device=""/>
-<part name="R24" library="CMU-ArtFab" deviceset="R-US_" device="R0805" value="100"/>
+<part name="R24" library="CMU-ArtFab" deviceset="R-US_" device="R0603" value="100"/>
 <part name="GND7" library="supply1" library_urn="urn:adsk.eagle:library:371" deviceset="GND" device=""/>
 <part name="GND8" library="supply1" library_urn="urn:adsk.eagle:library:371" deviceset="GND" device=""/>
+<part name="C12" library="adafruit" deviceset="C-US" device="C0805K" value="0.1uF"/>
+<part name="C10" library="adafruit" deviceset="C-US" device="C0805K" value="0.1uF"/>
 </parts>
 <sheets>
@@
 <instance part="U$7" gate="G$1" x="88.9" y="134.62"/>
 <instance part="U$9" gate="G$1" x="121.92" y="109.22" rot="MR0"/>
-<instance part="C10" gate="G$1" x="58.42" y="157.48" rot="R180"/>
 <instance part="R20" gate="G$1" x="66.04" y="165.1" rot="R180"/>
 <instance part="LED2" gate="G$1" x="121.92" y="175.26"/>
@@
 <instance part="P+1" gate="1" x="121.92" y="182.88"/>
 <instance part="P+4" gate="1" x="50.8" y="160.02"/>
-<instance part="C11" gate="G$1" x="114.3" y="137.16" rot="R180"/>
 <instance part="R23" gate="G$1" x="124.46" y="134.62" rot="R180"/>
 <instance part="U$12" gate="G$1" x="137.16" y="134.62" rot="R270"/>
@@
 <attribute name="VALUE" x="88.9" y="101.6" size="1.778" layer="96" ratio="12"/>
 </instance>
+<instance part="C12" gate="G$1" x="114.3" y="137.16" rot="R180"/>
+<instance part="C10" gate="G$1" x="58.42" y="157.48" rot="R180"/>
 </instances>
 <busses>
@@
 <pinref part="U$1" gate="G$1" pin="3GND"/>
 <wire x1="60.96" y1="160.02" x2="76.2" y2="160.02" width="0.1524" layer="91"/>
-<pinref part="C10" gate="G$1" pin="-"/>
 <wire x1="58.42" y1="162.56" x2="58.42" y2="167.64" width="0.1524" layer="91"/>
 <junction x="58.42" y="167.64"/>
+<pinref part="C10" gate="G$1" pin="2"/>
 </segment>
 </net>
@@
 <wire x1="50.8" y1="157.48" x2="50.8" y2="154.94" width="0.1524" layer="91"/>
 <junction x="50.8" y="154.94"/>
-<pinref part="C10" gate="G$1" pin="+"/>
+<pinref part="C10" gate="G$1" pin="1"/>
 <junction x="58.42" y="154.94"/>
 </segment>
@@
 <segment>
 <pinref part="U$7" gate="G$1" pin="5VCC"/>
-<pinref part="C11" gate="G$1" pin="+"/>
 <wire x1="106.68" y1="134.62" x2="114.3" y2="134.62" width="0.1524" layer="91"/>
 <pinref part="R23" gate="G$1" pin="2"/>
-<wire x1="119.38" y1="134.62" x2="114.3" y2="134.62" width="0.1524" layer="91"/>
+<pinref part="C12" gate="G$1" pin="1"/>
+<wire x1="114.3" y1="134.62" x2="119.38" y2="134.62" width="0.1524" layer="91"/>
 <junction x="114.3" y="134.62"/>
 </segment>
@@
 <segment>
 <pinref part="U$7" gate="G$1" pin="6GND"/>
-<pinref part="C11" gate="G$1" pin="-"/>
 <wire x1="106.68" y1="142.24" x2="114.3" y2="142.24" width="0.1524" layer="91"/>
+<pinref part="C12" gate="G$1" pin="2"/>
 </segment>
 </net>
@@
 <compatibility>
 <note version="8.2" severity="warning">
-Since Version 8.2, Eagle supports online libraries. The ids
+Since Version 8.2, EAGLE supports online libraries. The ids
 of those online libraries will not be understood (or retained)
 with this version.
