File: piezo-preamp-tickler-V0/piezo-preamp-tickler_V3-3_single-supply-OPA1642.brd (EAGLE design)
At the start: 114.3 x 18 mm, 62 parts, among them IC1 OPA2134UA, Q2 MMBFJ201, SW2-SPST INPUT-select

Commit message: piezo preamp fixes
Parts:
- IC1: value OPA2134UA -> OPA1642
Changed lines of the file:
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@@
 <attribute name="VALUE" x="92.188" y="4.148" size="1.27" layer="27" rot="R270"/>
 </element>
-<element name="IC1" library="linear" library_urn="urn:adsk.eagle:library:262" package="SO08" value="OPA2134UA" x="44.45" y="7.62" smashed="yes" rot="R270">
+<element name="IC1" library="linear" library_urn="urn:adsk.eagle:library:262" package="SO08" value="OPA1642" x="44.45" y="7.62" smashed="yes" rot="R270">
 <attribute name="NAME" x="42.545" y="10.287" size="0.8128" layer="25"/>
 </element>

Commit message: piezo preamp updates
Parts:
- L1: value (none) -> 100uH
Changed lines of the file:
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@@
 <element name="C4" library="adafruit" package="C0805K" value="0.1uF" x="0.254" y="-17.018"/>
 <element name="C6" library="microbuilder" package="EIA3216-18/A-R" value="100uF" x="3.048" y="-20.828"/>
-<element name="L1" library="rcl" library_urn="urn:adsk.eagle:library:334" package="L3225P" package3d_urn="urn:adsk.eagle:package:23479/1" value="" x="0.762" y="-25.908">
+<element name="L1" library="rcl" library_urn="urn:adsk.eagle:library:334" package="L3225P" package3d_urn="urn:adsk.eagle:package:23479/1" value="100uH" x="0.762" y="-25.908">
 <attribute name="SPICEPREFIX" value="L" x="0.762" y="-25.908" size="1.778" layer="27" display="off"/>
 </element>
