File: piezo-preamp-tickler-V0/piezo-preamp-tickler_V3-7_single-supply-OPA1642.sch (EAGLE design)
At the start: 61 parts, among them IC1 OPA1642, IC4 BQ297X, IC5 SC4503, IC6 TPS7A49, J1 HEADPHONES, J2 PHONE, J3 Mixer, J5 Battery, Q1 MMBFJ201, SW1 SWITCH_DPDT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

Commit message: Add files via upload
Parts:
- L2: device SparkFun-Passives:INDUCTOR30OHM,1.8A -> SparkFun-Passives:INDUCTORCR54
Connections:
- removed net N$15: C6.1, J4.VBUS, U$1.4VDD
- removed net V+: C10.1, C11.1, C15.1, D2.C, IC6.EN, IC6.IN, LED2.A, R18.2
- new net +5V: C6.1, J4.VBUS, LED2.A, U$1.4VDD
- new net VUSB: C10.1, C11.1, C15.1, D2.C, IC6.EN, IC6.IN, R18.2
Changed lines of the file:
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@@
 <part name="LED2" library="led" library_urn="urn:adsk.eagle:library:259" deviceset="LED" device="3MM" package3d_urn="urn:adsk.eagle:package:15797/1" value="Charge"/>
 <part name="R14" library="CMU-ArtFab" deviceset="R-US_" device="R0603" value="470"/>
-<part name="P+3" library="supply1" library_urn="urn:adsk.eagle:library:371" deviceset="V+" device=""/>
 <part name="R13" library="CMU-ArtFab" deviceset="R-US_" device="R0603" value="5k"/>
 <part name="IC4" library="CMU-ArtFab" deviceset="BQ297X-BATTERY-MANAGER" device="LONG" value="BQ297X"/>
@@
 <part name="GND4" library="supply1" library_urn="urn:adsk.eagle:library:371" deviceset="GND" device=""/>
 <part name="IC5" library="CMU-ArtFab" deviceset="SC4503" device=""/>
-<part name="L2" library="SparkFun-Passives" deviceset="INDUCTOR" device="30OHM,1.8A" value="2.7uH"/>
+<part name="L2" library="SparkFun-Passives" deviceset="INDUCTOR" device="CR54" value="2.7uH"/>
 <part name="J3" library="CMU-ArtFab" deviceset="TRS-1/8&quot;-3.5MM" device="" value="Mixer"/>
 <part name="J1" library="CMU-ArtFab" deviceset="TRRS-1/8&quot;-3.5MM" device="LGPADS" value="HEADPHONES"/>
@@
 <part name="R23" library="CMU-ArtFab" deviceset="R-US_" device="R0603" value="10M"/>
 <part name="C16" library="rcl" library_urn="urn:adsk.eagle:library:334" deviceset="C-EU" device="C0603" package3d_urn="urn:adsk.eagle:package:23616/2" value="4.7uF"/>
-<part name="P+2" library="supply1" library_urn="urn:adsk.eagle:library:371" deviceset="V+" device="" value="VUSB"/>
+<part name="P+2" library="supply1" library_urn="urn:adsk.eagle:library:371" deviceset="+5V" device="" value="VUSB"/>
+<part name="P+3" library="supply1" library_urn="urn:adsk.eagle:library:371" deviceset="+5V" device="" value="VUSB"/>
 </parts>
 <sheets>
@@
 <instance part="LED2" gate="G$1" x="129.54" y="182.88" rot="R270"/>
 <instance part="R14" gate="G$1" x="114.3" y="182.88" rot="R180"/>
-<instance part="P+3" gate="1" x="142.24" y="185.42"/>
 <instance part="R13" gate="G$1" x="50.8" y="182.88"/>
 <instance part="IC4" gate="G$1" x="119.38" y="142.24" rot="MR180"/>
@@
 <instance part="C16" gate="G$1" x="111.76" y="195.58"/>
 <instance part="P+2" gate="1" x="45.72" y="200.66"/>
+<instance part="P+3" gate="1" x="142.24" y="185.42"/>
 </instances>
 <busses>
@@
 </segment>
 </net>
-<net name="V+" class="0">
+<net name="VUSB" class="0">
 <segment>
 <wire x1="309.88" y1="175.26" x2="312.42" y2="175.26" width="0.1524" layer="91"/>
@@
 <wire x1="424.18" y1="182.88" x2="424.18" y2="170.18" width="0.1524" layer="91"/>
 <pinref part="C15" gate="G$1" pin="1"/>
-</segment>
-<segment>
-<pinref part="LED2" gate="G$1" pin="A"/>
-<pinref part="P+3" gate="1" pin="V+"/>
-<wire x1="142.24" y1="182.88" x2="132.08" y2="182.88" width="0.1524" layer="91"/>
 </segment>
 </net>
@@
 </segment>
 </net>
-<net name="N$15" class="0">
-<segment>
+<net name="+5V" class="0">
+<segment>
+<pinref part="J4" gate="G$1" pin="VBUS"/>
 <wire x1="45.72" y1="198.12" x2="45.72" y2="195.58" width="0.1524" layer="91"/>
-<pinref part="J4" gate="G$1" pin="VBUS"/>
 <wire x1="45.72" y1="195.58" x2="40.64" y2="195.58" width="0.1524" layer="91"/>
 <junction x="45.72" y="195.58"/>
 <pinref part="C6" gate="G$1" pin="1"/>
 <wire x1="48.26" y1="195.58" x2="45.72" y2="195.58" width="0.1524" layer="91"/>
+<junction x="48.26" y="195.58"/>
+<wire x1="48.26" y1="198.12" x2="48.26" y2="195.58" width="0.1524" layer="91"/>
 <pinref part="U$1" gate="G$1" pin="4VDD"/>
 <wire x1="58.42" y1="198.12" x2="48.26" y2="198.12" width="0.1524" layer="91"/>
-<wire x1="48.26" y1="198.12" x2="48.26" y2="195.58" width="0.1524" layer="91"/>
-<junction x="48.26" y="195.58"/>
-<pinref part="P+2" gate="1" pin="V+"/>
-</segment>
-</net>
+<pinref part="P+2" gate="1" pin="+5V"/>
+</segment>
+<segment>
+<pinref part="LED2" gate="G$1" pin="A"/>
+<wire x1="132.08" y1="182.88" x2="142.24" y2="182.88" width="0.1524" layer="91"/>
+<pinref part="P+3" gate="1" pin="+5V"/>
+</segment>
+</net>

Commit message: Add files via upload
Parts:
- IC1: value OPA1642 -> TL072D; device linear:OPA2134UA -> linear:TL072D
Connections:
- net GND: now also IC1P.V-; no longer IC1A.V-
- net N$8: now also IC1P.V+; no longer IC1A.V+

Commit message: Add files via upload
IC names changed according to convention
Parts:
- renumbered U$1 to IC2, U$2 to IC3
Changed lines of the file:
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@@
 <part name="C15" library="rcl" library_urn="urn:adsk.eagle:library:334" deviceset="C-EU" device="C0603" package3d_urn="urn:adsk.eagle:package:23616/2" value="10uF"/>
 <part name="R6" library="CMU-ArtFab" deviceset="POT" device="THUMBPOT14" value="50K"/>
-<part name="U$1" library="CMU-ArtFab" deviceset="MCP73831" device=""/>
+<part name="IC2" library="CMU-ArtFab" deviceset="MCP73831" device=""/>
 <part name="U2" library="microbuilder" deviceset="VBAT" device=""/>
-<part name="U$2" library="CMU-ArtFab" deviceset="QS6K1" device=""/>
+<part name="IC3" library="CMU-ArtFab" deviceset="QS6K1" device=""/>
 <part name="R15" library="CMU-ArtFab" deviceset="R-US_" device="R0603" value="2.2k"/>
 <part name="R22" library="CMU-ArtFab" deviceset="R-US_" device="R0603" value="10M"/>
@@
 <instance part="C14" gate="G$1" x="419.1" y="157.48"/>
 <instance part="C15" gate="G$1" x="434.34" y="165.1"/>
-<instance part="U$1" gate="G$1" x="81.28" y="190.5" rot="R180"/>
+<instance part="IC2" gate="G$1" x="81.28" y="190.5" rot="R180"/>
 <instance part="U2" gate="G$1" x="106.68" y="205.74"/>
-<instance part="U$2" gate="G$1" x="63.5" y="144.78" rot="MR0"/>
+<instance part="IC3" gate="G$1" x="63.5" y="144.78" rot="MR0"/>
 <instance part="R15" gate="G$1" x="157.48" y="127" rot="R90"/>
 <instance part="R22" gate="G$1" x="93.98" y="129.54" rot="R90"/>
@@
 </segment>
 <segment>
-<pinref part="U$2" gate="G$1" pin="2S2"/>
+<pinref part="IC3" gate="G$1" pin="2S2"/>
 <wire x1="83.82" y1="144.78" x2="91.44" y2="144.78" width="0.1524" layer="91"/>
 <wire x1="91.44" y1="144.78" x2="91.44" y2="119.38" width="0.1524" layer="91"/>
@@
 </segment>
 <segment>
-<pinref part="U$1" gate="G$1" pin="3VBAT"/>
+<pinref part="IC2" gate="G$1" pin="3VBAT"/>
 <pinref part="U2" gate="G$1" pin="VBAT"/>
 <wire x1="104.14" y1="198.12" x2="106.68" y2="198.12" width="0.1524" layer="91"/>
@@
 <pinref part="C7" gate="G$1" pin="1"/>
 <wire x1="38.1" y1="165.1" x2="38.1" y2="152.4" width="0.1524" layer="91"/>
-<pinref part="U$2" gate="G$1" pin="6D1"/>
+<pinref part="IC3" gate="G$1" pin="6D1"/>
 <wire x1="38.1" y1="152.4" x2="43.18" y2="152.4" width="0.1524" layer="91"/>
 </segment>
@@
 <net name="N$21" class="0">
 <segment>
-<pinref part="U$1" gate="G$1" pin="5PROG"/>
+<pinref part="IC2" gate="G$1" pin="5PROG"/>
 <pinref part="R13" gate="G$1" pin="2"/>
 <wire x1="55.88" y1="182.88" x2="58.42" y2="182.88" width="0.1524" layer="91"/>
@@
 <segment>
 <pinref part="R14" gate="G$1" pin="2"/>
-<pinref part="U$1" gate="G$1" pin="1STAT"/>
+<pinref part="IC2" gate="G$1" pin="1STAT"/>
 <wire x1="109.22" y1="182.88" x2="104.14" y2="182.88" width="0.1524" layer="91"/>
 </segment>
@@
 <net name="N$23" class="0">
 <segment>
-<pinref part="U$2" gate="G$1" pin="5S1"/>
-<pinref part="U$2" gate="G$1" pin="4D2"/>
+<pinref part="IC3" gate="G$1" pin="5S1"/>
+<pinref part="IC3" gate="G$1" pin="4D2"/>
 <wire x1="43.18" y1="144.78" x2="43.18" y2="137.16" width="0.1524" layer="91"/>
 </segment>
@@
 <net name="N$27" class="0">
 <segment>
-<pinref part="U$2" gate="G$1" pin="1G1"/>
+<pinref part="IC3" gate="G$1" pin="1G1"/>
 <wire x1="83.82" y1="152.4" x2="86.36" y2="152.4" width="0.1524" layer="91"/>
 <wire x1="86.36" y1="152.4" x2="91.44" y2="152.4" width="0.1524" layer="91"/>
@@
 <net name="N$31" class="0">
 <segment>
-<pinref part="U$2" gate="G$1" pin="3G2"/>
+<pinref part="IC3" gate="G$1" pin="3G2"/>
 <wire x1="83.82" y1="137.16" x2="93.98" y2="137.16" width="0.1524" layer="91"/>
 <pinref part="IC4" gate="G$1" pin="CHG-FET"/>
@@
 <pinref part="C16" gate="G$1" pin="2"/>
 <junction x="111.76" y="190.5"/>
-<pinref part="U$1" gate="G$1" pin="2VSS"/>
+<pinref part="IC2" gate="G$1" pin="2VSS"/>
 <wire x1="147.32" y1="190.5" x2="152.4" y2="190.5" width="0.1524" layer="91"/>
 <wire x1="104.14" y1="190.5" x2="111.76" y2="190.5" width="0.1524" layer="91"/>
@@
 <junction x="48.26" y="195.58"/>
 <wire x1="48.26" y1="198.12" x2="48.26" y2="195.58" width="0.1524" layer="91"/>
-<pinref part="U$1" gate="G$1" pin="4VDD"/>
+<pinref part="IC2" gate="G$1" pin="4VDD"/>
 <wire x1="58.42" y1="198.12" x2="48.26" y2="198.12" width="0.1524" layer="91"/>
 <pinref part="P+2" gate="1" pin="+5V"/>
