File: piezo-preamp-tickler-V0/piezo-preamp-tickler_V3-7_single-supply-TL072.sch (EAGLE design)
At the start: 61 parts, among them IC1 TL072D, IC2 MCP73831, IC3 QS6K1, IC4 BQ297X, IC5 SC4503, IC6 TPS7A49, J1 HEADPHONES, J2 PHONE, J3 Mixer, J5 Battery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

Commit message: moved IC6 in piezo preamp, routed jack signals on back side`
Parts:
- C2: device microbuilder:CAP_TANTALUMD/7343_REFLOW -> resistor:CPOL-EUC
- C5: device adafruit:C-USC0805 -> resistor:CPOL-EUB
Connections:
- net N$16: now also C5.-; no longer C5.2
- net N$6: now also C5.+; no longer C5.1
