File: MEMS-preamp/Lipo-Charger-12V-setup copy.brd (EAGLE design)
At the start: 33.6 x 19.9 mm, 7 parts

Commit message: chip/MOM updates
Other:
- board size 33.6 x 19.9 mm -> 33.6 x 20.6 mm
Changed lines of the file:
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@@
 <setting verticaltext="up"/>
 </settings>
-<grid distance="1" unitdist="mm" unit="mm" style="lines" multiple="1" display="no" altdistance="0.01" altunitdist="mm" altunit="mm"/>
+<grid distance="0.05" unitdist="inch" unit="inch" style="lines" multiple="1" display="no" altdistance="0.025" altunitdist="inch" altunit="inch"/>
 <layers>
 <layer number="1" name="Top" color="4" fill="1" visible="yes" active="yes"/>
@@
 <plain>
 <wire x1="0" y1="0" x2="33.635" y2="0" width="0" layer="20"/>
-<wire x1="33.635" y1="0" x2="33.635" y2="19.863" width="0" layer="20"/>
-<wire x1="33.635" y1="19.863" x2="0" y2="19.863" width="0" layer="20"/>
-<wire x1="0" y1="19.863" x2="0" y2="0" width="0" layer="20"/>
+<wire x1="33.635" y1="0" x2="33.635" y2="20.625" width="0" layer="20"/>
+<wire x1="33.635" y1="20.625" x2="0" y2="20.625" width="0" layer="20"/>
+<wire x1="0" y1="20.625" x2="0" y2="0" width="0" layer="20"/>
 </plain>
 <attributes>
