File: MEMS-preamp/Lipo-Charger-12V-setup.sch (EAGLE design)
At the start: 7 parts

Commit message: chip/MOM updates
Parts:
- removed OUT: (no value), CMU-ArtFab:M02LOCK
- added BAT1: (no value), Daniel:BATTERYA23
- R6: device CMU-ArtFab:R-US_0204/5 -> CMU-ArtFab:R-US_0204/7
Connections:
- net +12V: now also BAT1.+; no longer OUT.1
- net GND: now also BAT1.-; no longer OUT.2
- net N$1: now also POWER.1; no longer POWER.3
Other:
- moved on the sheet: LED1, R6
Changed lines of the file:
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@@
 <part name="LED1" library="led" deviceset="LED" device="3MM"/>
 <part name="GND1" library="supply1" deviceset="GND" device=""/>
-<part name="R6" library="CMU-ArtFab" deviceset="R-US_" device="0204/5" value="390"/>
+<part name="R6" library="CMU-ArtFab" deviceset="R-US_" device="0204/7" value="390"/>
 <part name="J_REG_12V" library="CMU-ArtFab" deviceset="POLOLU_VOLTAGE_REGULATORS_3PIN" device="" value="POLOLU_VOLTAGE_REGULATORS_3PIN"/>
 <part name="GND12" library="supply1" deviceset="GND" device=""/>
@@
 <part name="U$3" library="microbuilder" deviceset="VIN" device=""/>
 <part name="BATTERY" library="CMU-ArtFab" deviceset="M02" device="LOCK"/>
-<part name="OUT" library="CMU-ArtFab" deviceset="M02" device="LOCK"/>
-<part name="P+2" library="supply1" deviceset="+12V" device=""/>
-<part name="GND2" library="supply1" deviceset="GND" device=""/>
+<part name="BAT1" library="Daniel" deviceset="BATTERY" device="A23"/>
+<part name="P+3" library="supply1" deviceset="+12V" device=""/>
+<part name="GND3" library="supply1" deviceset="GND" device=""/>
 </parts>
 <sheets>
@@
 </plain>
 <instances>
-<instance part="LED1" gate="G$1" x="48.26" y="58.42"/>
+<instance part="LED1" gate="G$1" x="48.26" y="60.96"/>
 <instance part="GND1" gate="1" x="48.26" y="43.18" smashed="yes">
 <attribute name="VALUE" x="45.72" y="40.64" size="1.778" layer="96" ratio="12"/>
 </instance>
-<instance part="R6" gate="G$1" x="48.26" y="68.58" rot="R90"/>
+<instance part="R6" gate="G$1" x="48.26" y="78.74" rot="R90"/>
 <instance part="J_REG_12V" gate="J_REG_5V" x="7.62" y="40.64"/>
 <instance part="GND12" gate="1" x="7.62" y="20.32" smashed="yes">
@@
 <instance part="POWER" gate="G$1" x="17.78" y="73.66"/>
 <instance part="U$17" gate="G$1" x="10.16" y="88.9"/>
-<instance part="U$16" gate="G$1" x="48.26" y="81.28"/>
+<instance part="U$16" gate="G$1" x="48.26" y="91.44"/>
 <instance part="U$3" gate="G$1" x="-15.24" y="50.8"/>
 <instance part="BATTERY" gate="G$1" x="35.56" y="78.74" rot="R180"/>
-<instance part="OUT" gate="G$1" x="81.28" y="50.8" rot="R180"/>
-<instance part="P+2" gate="1" x="68.58" y="55.88"/>
-<instance part="GND2" gate="1" x="66.04" y="43.18" smashed="yes">
-<attribute name="VALUE" x="63.5" y="40.64" size="1.778" layer="96" ratio="12"/>
+<instance part="BAT1" gate="G$1" x="73.66" y="68.58"/>
+<instance part="P+3" gate="1" x="63.5" y="73.66"/>
+<instance part="GND3" gate="1" x="86.36" y="66.04" smashed="yes">
+<attribute name="VALUE" x="83.82" y="63.5" size="1.778" layer="96" ratio="12"/>
 </instance>
 </instances>
@@
 <nets>
 <net name="GND" class="0">
-<segment>
-<pinref part="LED1" gate="G$1" pin="C"/>
-<pinref part="GND1" gate="1" pin="GND"/>
-<wire x1="48.26" y1="53.34" x2="48.26" y2="45.72" width="0.1524" layer="91"/>
-</segment>
 <segment>
 <pinref part="J_REG_12V" gate="J_REG_5V" pin="GND"/>
@@
 </segment>
 <segment>
-<pinref part="OUT" gate="G$1" pin="2"/>
-<pinref part="GND2" gate="1" pin="GND"/>
-<wire x1="73.66" y1="48.26" x2="66.04" y2="48.26" width="0.1524" layer="91"/>
-<wire x1="66.04" y1="48.26" x2="66.04" y2="45.72" width="0.1524" layer="91"/>
+<pinref part="BAT1" gate="G$1" pin="-"/>
+<pinref part="GND3" gate="1" pin="GND"/>
+<wire x1="78.74" y1="68.58" x2="86.36" y2="68.58" width="0.1524" layer="91"/>
+</segment>
+<segment>
+<pinref part="LED1" gate="G$1" pin="C"/>
+<pinref part="GND1" gate="1" pin="GND"/>
+<wire x1="48.26" y1="55.88" x2="48.26" y2="45.72" width="0.1524" layer="91"/>
 </segment>
 </net>
@@
 </segment>
 <segment>
-<wire x1="48.26" y1="78.74" x2="48.26" y2="73.66" width="0.1524" layer="91"/>
-<pinref part="R6" gate="G$1" pin="2"/>
-<pinref part="U$16" gate="G$1" pin="VIN"/>
-</segment>
-<segment>
 <pinref part="J_REG_12V" gate="J_REG_5V" pin="VIN"/>
 <wire x1="-15.24" y1="48.26" x2="-15.24" y2="40.64" width="0.1524" layer="91"/>
@@
 <pinref part="U$3" gate="G$1" pin="VIN"/>
 </segment>
-</net>
-<net name="N$16" class="0">
 <segment>
-<pinref part="R6" gate="G$1" pin="1"/>
-<pinref part="LED1" gate="G$1" pin="A"/>
-<wire x1="48.26" y1="63.5" x2="48.26" y2="60.96" width="0.1524" layer="91"/>
+<pinref part="U$16" gate="G$1" pin="VIN"/>
+<pinref part="R6" gate="G$1" pin="2"/>
+<wire x1="48.26" y1="88.9" x2="48.26" y2="83.82" width="0.1524" layer="91"/>
 </segment>
 </net>
@@
 </segment>
 <segment>
-<pinref part="OUT" gate="G$1" pin="1"/>
-<pinref part="P+2" gate="1" pin="+12V"/>
-<wire x1="73.66" y1="50.8" x2="68.58" y2="50.8" width="0.1524" layer="91"/>
-<wire x1="68.58" y1="50.8" x2="68.58" y2="53.34" width="0.1524" layer="91"/>
+<pinref part="BAT1" gate="G$1" pin="+"/>
+<pinref part="P+3" gate="1" pin="+12V"/>
+<wire x1="68.58" y1="68.58" x2="63.5" y2="68.58" width="0.1524" layer="91"/>
+<wire x1="63.5" y1="68.58" x2="63.5" y2="71.12" width="0.1524" layer="91"/>
 </segment>
 </net>
@@
 <net name="N$1" class="0">
 <segment>
-<pinref part="POWER" gate="G$1" pin="3"/>
 <pinref part="BATTERY" gate="G$1" pin="2"/>
-<wire x1="22.86" y1="71.12" x2="27.94" y2="71.12" width="0.1524" layer="91"/>
-<wire x1="27.94" y1="71.12" x2="27.94" y2="76.2" width="0.1524" layer="91"/>
+<pinref part="POWER" gate="G$1" pin="1"/>
+<wire x1="27.94" y1="76.2" x2="22.86" y2="76.2" width="0.1524" layer="91"/>
 </segment>
 </net>
+<net name="N$2" class="0">
+<segment>
+<pinref part="R6" gate="G$1" pin="1"/>
+<pinref part="LED1" gate="G$1" pin="A"/>
+<wire x1="48.26" y1="73.66" x2="48.26" y2="63.5" width="0.1524" layer="91"/>
+</segment>
+</net>
