File: MEMS-preamp/ICS40300-Silicon-Mic_Rev-A.sch (EAGLE design)
At the start: 10 parts, among them U2 MIC5225-3.3

Commit message: Mems Board Updates
Parts:
- removed FID1, FID2: FIDUCIAL"", microbuilder:FIDUCIAL""
- added C5: 10uF, microbuilder:CAP_CERAMIC0805-NOOUTLINE
- added R1: (no value), adafruit:R-US_M0805
- C1: value 10uF -> (none); device microbuilder:CAP_CERAMIC0805-NOOUTLINE -> adafruit:C-USC3216
Connections:
- new net N$3: C5.1, R1.1
- net GND: now also R1.2
- net N$1: now also C1.1, C5.2; no longer C1.2
- net N$2: now also C1.2; no longer C1.1
Other:
- moved on the sheet: C1, JP1
