File: MEMS-preamp/ICS40300-Silicon-Mic_Rev-D.sch (EAGLE design)
At the start: 8 parts, among them U1 ICS-40300, U2 MIC5225-3.3

Commit message: piezo preamp updates
Other:
- moved on the sheet: C3, C4, U2
