File: MEMS-preamp/MEMS-preamp_v05.sch (EAGLE design)
At the start: 19 parts, among them Q1 OPA2134

Commit message: piezo preamp updates
Parts:
- removed BATTERY: (no value), SparkFun-Connectors:CONN_02LOCK
- removed J_REG_12V: POLOLU_VOLTAGE_REGULATORS_3PIN, CMU-ArtFab:POLOLU_VOLTAGE_REGULATORS_3PIN
- removed LED1: (no value), led:LED3MM
- removed POWER: SPDT, CMU-ArtFab:SWITCH_SPDTTE-CONNECT
- removed R10: 390, CMU-ArtFab:R-US_0204/5
- removed USB-LIPO-CHARGER: TP4056-MODULE, CMU-ArtFab:TP4056-MODULE
Connections:
- removed net N$16: LED1.A, R10.1
- removed net N$18: BATTERY.1, USB-LIPO-CHARGER.B+
- removed net N$19: POWER.2, USB-LIPO-CHARGER.B-
- removed net N$2: BATTERY.2, POWER.1
- removed net VBAT: J_REG_12V.VIN, R10.2, USB-LIPO-CHARGER.OUT+
- net +12V: no longer J_REG_12V.VOUT
- net GND: no longer J_REG_12V.GND, LED1.C, USB-LIPO-CHARGER.OUT-
- net N$10: now also POT1/2.S; no longer POT1/2.A
- net N$9: now also POT1/1.S; no longer POT1/1.A
Other:
- note removed: "Battery Charging"
- note removed: "Power LED"
- note removed: "Voltage Regulation"
- moved on the sheet: POT1/2
Changed lines of the file:
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@@
 <part name="U$1" library="CMU-ArtFab" deviceset="1/8&quot;-F-STEREO-PCB" device=""/>
 <part name="GND10" library="supply1" deviceset="GND" device=""/>
-<part name="LED1" library="led" deviceset="LED" device="3MM"/>
-<part name="GND1" library="supply1" deviceset="GND" device=""/>
-<part name="R10" library="CMU-ArtFab" deviceset="R-US_" device="0204/5" value="390"/>
-<part name="J_REG_12V" library="CMU-ArtFab" deviceset="POLOLU_VOLTAGE_REGULATORS_3PIN" device="" value="POLOLU_VOLTAGE_REGULATORS_3PIN"/>
-<part name="GND12" library="supply1" deviceset="GND" device=""/>
-<part name="U$2" library="microbuilder" deviceset="VBAT" device=""/>
-<part name="P+1" library="supply1" deviceset="+12V" device=""/>
-<part name="U$3" library="microbuilder" deviceset="VBAT" device=""/>
 <part name="P+5" library="supply1" deviceset="+12V" device=""/>
-<part name="USB-LIPO-CHARGER" library="CMU-ArtFab" deviceset="TP4056-MODULE" device=""/>
-<part name="U$8" library="microbuilder" deviceset="VBAT" device=""/>
-<part name="GND13" library="supply1" deviceset="GND" device=""/>
 <part name="P+6" library="supply1" deviceset="+12V" device=""/>
-<part name="POWER" library="CMU-ArtFab" deviceset="SWITCH_SPDT" device="TE-CONNECT" value="SPDT"/>
 <part name="P+2" library="supply1" deviceset="+12V" device=""/>
-<part name="BATTERY" library="SparkFun-Connectors" deviceset="CONN_02" device="LOCK"/>
 <part name="R3" library="CMU-ArtFab" deviceset="R-US_" device="0204/5" value="1k"/>
 <part name="C2" library="rcl" deviceset="CPOL-EU" device="E2.5-5" value="10u"/>
@@
 <sheet>
 <plain>
-<text x="109.22" y="38.1" size="1.778" layer="91">Voltage Regulation</text>
-<text x="38.1" y="38.1" size="1.778" layer="91">Battery Charging</text>
-<text x="177.8" y="38.1" size="1.778" layer="91">Power LED</text>
 </plain>
 <instances>
@@
 <attribute name="VALUE" x="182.88" y="58.42" size="1.778" layer="96" ratio="12"/>
 </instance>
-<instance part="LED1" gate="G$1" x="185.42" y="7.62"/>
-<instance part="GND1" gate="1" x="185.42" y="-2.54" smashed="yes">
-<attribute name="VALUE" x="182.88" y="-5.08" size="1.778" layer="96" ratio="12"/>
-</instance>
-<instance part="R10" gate="G$1" x="185.42" y="17.78" rot="R90"/>
-<instance part="J_REG_12V" gate="J_REG_5V" x="119.38" y="20.32"/>
-<instance part="GND12" gate="1" x="119.38" y="0" smashed="yes">
-<attribute name="VALUE" x="116.84" y="-2.54" size="1.778" layer="96" ratio="12"/>
-</instance>
-<instance part="U$2" gate="G$1" x="96.52" y="25.4"/>
-<instance part="P+1" gate="1" x="144.78" y="27.94"/>
-<instance part="U$3" gate="G$1" x="185.42" y="30.48"/>
 <instance part="P+5" gate="1" x="109.22" y="119.38"/>
-<instance part="USB-LIPO-CHARGER" gate="G$1" x="33.02" y="15.24"/>
-<instance part="U$8" gate="G$1" x="48.26" y="27.94"/>
-<instance part="GND13" gate="1" x="48.26" y="5.08" smashed="yes">
-<attribute name="VALUE" x="45.72" y="2.54" size="1.778" layer="96" ratio="12"/>
-</instance>
 <instance part="P+6" gate="1" x="38.1" y="114.3"/>
-<instance part="POWER" gate="G$1" x="55.88" y="12.7"/>
 <instance part="P+2" gate="1" x="22.86" y="81.28"/>
-<instance part="BATTERY" gate="G$1" x="73.66" y="17.78" rot="R180"/>
 <instance part="R3" gate="G$1" x="119.38" y="71.12"/>
 <instance part="C2" gate="G$1" x="165.1" y="71.12" smashed="yes" rot="R90">
@@
 </instance>
 <instance part="POT1" gate="/1" x="81.28" y="50.8" rot="R90"/>
-<instance part="POT1" gate="/2" x="147.32" y="53.34" rot="R90"/>
+<instance part="POT1" gate="/2" x="157.48" y="53.34" rot="R90"/>
 </instances>
 <busses>
@@
 <wire x1="190.5" y1="66.04" x2="185.42" y2="66.04" width="0.1524" layer="91"/>
 <wire x1="185.42" y1="66.04" x2="185.42" y2="63.5" width="0.1524" layer="91"/>
-</segment>
-<segment>
-<pinref part="LED1" gate="G$1" pin="C"/>
-<pinref part="GND1" gate="1" pin="GND"/>
-<wire x1="185.42" y1="2.54" x2="185.42" y2="0" width="0.1524" layer="91"/>
-</segment>
-<segment>
-<pinref part="J_REG_12V" gate="J_REG_5V" pin="GND"/>
-<pinref part="GND12" gate="1" pin="GND"/>
-<wire x1="119.38" y1="7.62" x2="119.38" y2="2.54" width="0.1524" layer="91"/>
-</segment>
-<segment>
-<pinref part="USB-LIPO-CHARGER" gate="G$1" pin="OUT-"/>
-<pinref part="GND13" gate="1" pin="GND"/>
-<wire x1="45.72" y1="10.16" x2="48.26" y2="10.16" width="0.1524" layer="91"/>
-<wire x1="48.26" y1="10.16" x2="48.26" y2="7.62" width="0.1524" layer="91"/>
 </segment>
 </net>
@@
 </segment>
 </net>
-<net name="VBAT" class="0">
-<segment>
-<pinref part="U$2" gate="G$1" pin="VBAT"/>
-<pinref part="J_REG_12V" gate="J_REG_5V" pin="VIN"/>
-<wire x1="96.52" y1="22.86" x2="96.52" y2="20.32" width="0.1524" layer="91"/>
-<wire x1="96.52" y1="20.32" x2="104.14" y2="20.32" width="0.1524" layer="91"/>
-</segment>
-<segment>
-<pinref part="R10" gate="G$1" pin="2"/>
-<pinref part="U$3" gate="G$1" pin="VBAT"/>
-<wire x1="185.42" y1="22.86" x2="185.42" y2="27.94" width="0.1524" layer="91"/>
-</segment>
-<segment>
-<pinref part="USB-LIPO-CHARGER" gate="G$1" pin="OUT+"/>
-<pinref part="U$8" gate="G$1" pin="VBAT"/>
-<wire x1="45.72" y1="20.32" x2="48.26" y2="20.32" width="0.1524" layer="91"/>
-<wire x1="48.26" y1="20.32" x2="48.26" y2="25.4" width="0.1524" layer="91"/>
-</segment>
-</net>
 <net name="N$9" class="0">
 <segment>
 <pinref part="Q1" gate="A" pin="OUT"/>
 <pinref part="C1" gate="G$1" pin="+"/>
-<wire x1="76.2" y1="71.12" x2="88.9" y2="71.12" width="0.1524" layer="91"/>
-<pinref part="POT1" gate="/1" pin="A"/>
-<wire x1="88.9" y1="71.12" x2="96.52" y2="71.12" width="0.1524" layer="91"/>
-<wire x1="88.9" y1="50.8" x2="88.9" y2="71.12" width="0.1524" layer="91"/>
-<junction x="88.9" y="71.12"/>
+<wire x1="76.2" y1="71.12" x2="81.28" y2="71.12" width="0.1524" layer="91"/>
+<pinref part="POT1" gate="/1" pin="S"/>
+<wire x1="81.28" y1="71.12" x2="96.52" y2="71.12" width="0.1524" layer="91"/>
+<wire x1="81.28" y1="55.88" x2="81.28" y2="71.12" width="0.1524" layer="91"/>
+<junction x="81.28" y="71.12"/>
 </segment>
 </net>
@@
 </segment>
 </net>
-<net name="N$16" class="0">
-<segment>
-<pinref part="R10" gate="G$1" pin="1"/>
-<pinref part="LED1" gate="G$1" pin="A"/>
-<wire x1="185.42" y1="12.7" x2="185.42" y2="10.16" width="0.1524" layer="91"/>
-</segment>
-</net>
 <net name="+12V" class="0">
-<segment>
-<pinref part="J_REG_12V" gate="J_REG_5V" pin="VOUT"/>
-<wire x1="134.62" y1="20.32" x2="144.78" y2="20.32" width="0.1524" layer="91"/>
-<wire x1="144.78" y1="20.32" x2="144.78" y2="25.4" width="0.1524" layer="91"/>
-<pinref part="P+1" gate="1" pin="+12V"/>
-</segment>
 <segment>
 <pinref part="R9" gate="G$1" pin="2"/>
@@
 </segment>
 </net>
-<net name="N$18" class="0">
-<segment>
-<pinref part="USB-LIPO-CHARGER" gate="G$1" pin="B+"/>
-<wire x1="45.72" y1="17.78" x2="66.04" y2="17.78" width="0.1524" layer="91"/>
-<pinref part="BATTERY" gate="G$1" pin="1"/>
-</segment>
-</net>
-<net name="N$19" class="0">
-<segment>
-<pinref part="USB-LIPO-CHARGER" gate="G$1" pin="B-"/>
-<wire x1="50.8" y1="12.7" x2="45.72" y2="12.7" width="0.1524" layer="91"/>
-<pinref part="POWER" gate="G$1" pin="2"/>
-</segment>
-</net>
-<net name="N$2" class="0">
-<segment>
-<pinref part="POWER" gate="G$1" pin="1"/>
-<wire x1="60.96" y1="15.24" x2="66.04" y2="15.24" width="0.1524" layer="91"/>
-<pinref part="BATTERY" gate="G$1" pin="2"/>
-</segment>
-</net>
 <net name="N$4" class="0">
 <segment>
@@
 <pinref part="Q1" gate="B" pin="OUT"/>
 <pinref part="C2" gate="G$1" pin="+"/>
-<wire x1="162.56" y1="71.12" x2="154.94" y2="71.12" width="0.1524" layer="91"/>
-<pinref part="POT1" gate="/2" pin="A"/>
-<wire x1="154.94" y1="71.12" x2="152.4" y2="71.12" width="0.1524" layer="91"/>
-<wire x1="154.94" y1="53.34" x2="154.94" y2="71.12" width="0.1524" layer="91"/>
-<junction x="154.94" y="71.12"/>
+<wire x1="162.56" y1="71.12" x2="157.48" y2="71.12" width="0.1524" layer="91"/>
+<pinref part="POT1" gate="/2" pin="S"/>
+<wire x1="157.48" y1="71.12" x2="152.4" y2="71.12" width="0.1524" layer="91"/>
+<wire x1="157.48" y1="58.42" x2="157.48" y2="71.12" width="0.1524" layer="91"/>
+<junction x="157.48" y="71.12"/>
 </segment>
 </net>
@@
 <wire x1="129.54" y1="68.58" x2="134.62" y2="68.58" width="0.1524" layer="91"/>
 <wire x1="134.62" y1="68.58" x2="137.16" y2="68.58" width="0.1524" layer="91"/>
-<wire x1="139.7" y1="53.34" x2="134.62" y2="53.34" width="0.1524" layer="91"/>
+<wire x1="149.86" y1="53.34" x2="134.62" y2="53.34" width="0.1524" layer="91"/>
 <wire x1="134.62" y1="53.34" x2="134.62" y2="68.58" width="0.1524" layer="91"/>
 <junction x="134.62" y="68.58"/>
