File: MEMS-preamp/MEMS-preamp_v06_Labels.sch (EAGLE design)
At the start: 45 parts, among them J1 Battery, Q1 OPA2134, Q2 BQ21040, Q5 BQ297X, Q7 DMN2400, SW1 SPDT

Commit message: updates to MEMS preamp /Users/ali/Documents/Development/eagle/MEMS-preamp/MEMS-preamp_v06_Labels.sch
Parts:
- removed C16: 68uF, SparkFun:CAP_POL3528
- removed C17: 2.2pf, adafruit:C-USC0805
- removed C18: 56nf, adafruit:C-USC0805
- removed C21, C23: 10nF, adafruit:C-USC0805
- removed C22, C24: 10uF, adafruit:C-USC0805
- removed LED4: (no value), led:LED3MM
- removed Q1: OPA2134, linear:OPA2134UA
- removed R26: 91.2k, CMU-ArtFab:R-US_R0603
- removed R27: 100k, CMU-ArtFab:R-US_R0603
- removed SC1: VREG12_SOT23-5, CMU-ArtFab:VREG12_SOT23-5
- removed U$13: TPS7A49, CMU-ArtFab:TPS7A49
- removed U$3: AUDIO-JACK3LGPADS, CMU-ArtFab:AUDIO-JACK3LGPADS
- added C10, C11, C14: 10uF, adafruit:C-USC0603
- added C12: 10uF, adafruit:C-USC0805
- added C13: 100u, rcl:CPOL-EUCT7343
- added C8, C9: 10nF, adafruit:C-USC0603
- added IC4: SC4503, CMU-ArtFab:SC4503
- added IC5: TPS7A49, CMU-ArtFab:TPS7A49
- added IC6: OPA2134, linear:OPA2134UA
- added J3: TRS-1/8"-3.5MM, CMU-ArtFab:TRS-1/8"-3.5MM
- added LED1: (no value), led:LED3MM
- added R14: 10, CMU-ArtFab:R-US_R0603
- added R15: 1k, CMU-ArtFab:R-US_R0603
- C2: value 10uF -> 0.1uF
- C3: device adafruit:C-USC0805 -> adafruit:C-USC0603
- C4: value 100u -> 56nf; device rcl:CPOL-EUCT7343 -> adafruit:C-USC0603
- C5: value 10uF -> 2.2pf; device adafruit:C-USC0805K -> adafruit:C-USC0603
- C6: value 10uF -> 68uF; device adafruit:C-USC0805 -> SparkFun:CAP_POL3528
- C7: value 0.1uF -> 10uF; device adafruit:C-USC0805K -> adafruit:C-USC0603
- J1: value Battery -> (none); device SparkFun-Connectors:CONN_02LOCK -> SparkFun-Connectors:USB_MICRO-BREDUCED_PASTE
- J2: value (none) -> Battery; device SparkFun-Connectors:USB_MICRO-BREDUCED_PASTE -> SparkFun-Connectors:CONN_02LOCK
- JP1: value Adafruit-SPW2430 -> ICS30400
- L1: value 2.7uH -> 2.7mH; device SparkFun:INDUCTORCR54 -> SparkFun-Passives:INDUCTORCR54-KIT
- R1: value 1k -> 390
- R11: value 10k -> 150k; device CMU-ArtFab:R-US_R0805 -> CMU-ArtFab:R-US_R0603
- R12: value 330 -> 150k; device CMU-ArtFab:R-US_R0805 -> CMU-ArtFab:R-US_R0603
- R13: value 15k -> 1k
- R2: value 1k -> 10k; device CMU-ArtFab:R-US_R0805 -> CMU-ArtFab:R-US_R0603
- R4: device CMU-ArtFab:R-US_R0805 -> CMU-ArtFab:R-US_R0603
- R5: value 390 -> 330; device CMU-ArtFab:R-US_R0805 -> CMU-ArtFab:R-US_R0603
- R6: value 1M -> 15k
- R7: value 150k -> 1M
- R8: value 150k -> 100k
- R9: value 10 -> 91.2k
- renumbered Q2 to IC2, Q5 to IC3, Q7 to IC1
Connections:
- net +12V: now also C7.1, C8.1, IC5.OUT, R11.2, R14.2, R9.1; no longer C21.1, C22.1, R26.1, R8.2, R9.2, U$13.OUT
- net GND: now also C10.2, C11.2, C13.-, C3.2, C4.2, C6.-, C7.2, C9.2, IC5.GND, IC6A.V-, J3.SLEEVE, LED1.C, R10.2, R12.1, R8.1; no longer C1.2, C16.-, C18.2, C22.2, C23.2, C24.2, C4.-, C6.2, LED4.C, Q1A.V-, R10.1, R27.2, R7.1, SC1.GND, U$13.GND, U$3.EARTH
- net GND2: now also C1.2, C2.2, J1.GND, R2.1; no longer C5.2, C7.2, J2.GND, R11.1
- net GROU[: now also IC6B.-IN, R15.2; no longer Q1B.-IN, R3.2
- net N$1: now also C13.+, IC6A.V+, R14.1; no longer C4.+, Q1A.V+, R9.1
- net N$10: now also C14.1, IC6B.OUT; no longer C2.1, Q1B.OUT
- net N$11: now also R3.1; no longer R2.1
- net N$12: now also IC4.SW; no longer SC1.SW
- net N$13: now also C4.1, IC4.SHDN, R6.1; no longer C18.1, R13.1, SC1.SHDN
- net N$14: now also C5.2, IC4.FB, R7.1, R8.2; no longer C17.2, R10.2, R6.1, SC1.FB
- net N$15: now also R3.2; no longer R2.2
- net N$17: now also R2.2; no longer R11.2
- net N$18: now also C2.1, R5.2; no longer C7.1, R12.2
- net N$2: now also LED1.A, R1.1; no longer LED4.A, R5.1
- net N$3: now also R13.1; no longer R1.1
- net N$4: now also C12.2, R15.1; no longer C3.2, R3.1
- net N$47: now also C8.2, IC5.FB, R10.1, R9.2; no longer C21.2, R26.2, R27.1, U$13.FB
- net N$48: now also C9.1, IC5.NR/SS; no longer C23.1, U$13.NR/SS
- net N$5: now also IC6A.-IN, R13.2; no longer Q1A.-IN, R1.2
- net N$6: now also J2.2; no longer J1.2
- net N$7: now also C14.2, J3.RING1, J3.TIP; no longer C2.2, U$3.RING1, U$3.TIP
- net N$8: now also C11.1, IC6A.+IN, IC6B.+IN, R11.1, R12.2; no longer C1.1, Q1A.+IN, Q1B.+IN, R7.2, R8.1
- net N$9: now also C12.1, IC6A.OUT; no longer C3.1, Q1A.OUT
- net V+: now also C1.1, C10.1, C6.+, IC5.EN, IC5.IN, J1.VBUS, R7.2; no longer C16.+, C17.1, C24.1, J2.VBUS, R6.2, U$13.EN, U$13.IN
- net VBAT: now also C3.1, IC4.IN, J2.1, R1.2, R5.1, R6.2; no longer C6.1, J1.1, R12.1, R13.2, R5.2, SC1.IN
Other:
- moved on the sheet: C1, C2, C3, C5, C7, D1, JP1, L1, POT1/1, POT1/2, R1, R10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
