File: MEMS-preamp/MEMS-preamp_v08.sch (EAGLE design)
At the start: 45 parts, among them IC1 DMN2400, IC2 BQ21040, IC3 BQ297X, IC4 SC4503, IC5 TPS7A49, IC6 OPA2134, J2 Battery, J3 TRS-1/8"-3.5MM, SW1 SPDT

Commit message: Vin of ICS40300 changed back to 12V pin for now
Connections:
- net +12V: now also JP1.1
- net V+: no longer JP1.1
Changed lines of the file:
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@@
 <grid distance="0.1" unitdist="inch" unit="inch" style="lines" multiple="1" display="no" altdistance="0.01" altunitdist="inch" altunit="inch"/>
 <layers>
-<layer number="1" name="Top" color="4" fill="1" visible="yes" active="no"/>
-<layer number="2" name="Route2" color="1" fill="3" visible="yes" active="no"/>
-<layer number="3" name="Route3" color="4" fill="3" visible="yes" active="no"/>
-<layer number="4" name="Route4" color="1" fill="4" visible="yes" active="no"/>
-<layer number="5" name="Route5" color="4" fill="4" visible="yes" active="no"/>
-<layer number="6" name="Route6" color="1" fill="8" visible="yes" active="no"/>
-<layer number="7" name="Route7" color="4" fill="8" visible="yes" active="no"/>
-<layer number="8" name="Route8" color="1" fill="2" visible="yes" active="no"/>
-<layer number="9" name="Route9" color="4" fill="2" visible="yes" active="no"/>
-<layer number="10" name="Route10" color="1" fill="7" visible="yes" active="no"/>
-<layer number="11" name="Route11" color="4" fill="7" visible="yes" active="no"/>
-<layer number="12" name="Route12" color="1" fill="5" visible="yes" active="no"/>
-<layer number="13" name="Route13" color="4" fill="5" visible="yes" active="no"/>
-<layer number="14" name="Route14" color="1" fill="6" visible="yes" active="no"/>
-<layer number="15" name="Route15" color="4" fill="6" visible="yes" active="no"/>
-<layer number="16" name="Bottom" color="1" fill="1" visible="yes" active="no"/>
-<layer number="17" name="Pads" color="2" fill="1" visible="yes" active="no"/>
-<layer number="18" name="Vias" color="2" fill="1" visible="yes" active="no"/>
-<layer number="19" name="Unrouted" color="6" fill="1" visible="yes" active="no"/>
-<layer number="20" name="Dimension" color="15" fill="1" visible="yes" active="no"/>
-<layer number="21" name="tPlace" color="7" fill="1" visible="yes" active="no"/>
-<layer number="22" name="bPlace" color="7" fill="1" visible="yes" active="no"/>
-<layer number="23" name="tOrigins" color="15" fill="1" visible="yes" active="no"/>
-<layer number="24" name="bOrigins" color="15" fill="1" visible="yes" active="no"/>
-<layer number="25" name="tNames" color="7" fill="1" visible="yes" active="no"/>
-<layer number="26" name="bNames" color="7" fill="1" visible="yes" active="no"/>
-<layer number="27" name="tValues" color="7" fill="1" visible="yes" active="no"/>
-<layer number="28" name="bValues" color="7" fill="1" visible="yes" active="no"/>
+<layer number="1" name="Top" color="4" fill="1" visible="no" active="no"/>
+<layer number="2" name="Route2" color="1" fill="3" visible="no" active="no"/>
+<layer number="3" name="Route3" color="4" fill="3" visible="no" active="no"/>
+<layer number="4" name="Route4" color="1" fill="4" visible="no" active="no"/>
+<layer number="5" name="Route5" color="4" fill="4" visible="no" active="no"/>
+<layer number="6" name="Route6" color="1" fill="8" visible="no" active="no"/>
+<layer number="7" name="Route7" color="4" fill="8" visible="no" active="no"/>
+<layer number="8" name="Route8" color="1" fill="2" visible="no" active="no"/>
+<layer number="9" name="Route9" color="4" fill="2" visible="no" active="no"/>
+<layer number="10" name="Route10" color="1" fill="7" visible="no" active="no"/>
+<layer number="11" name="Route11" color="4" fill="7" visible="no" active="no"/>
+<layer number="12" name="Route12" color="1" fill="5" visible="no" active="no"/>
+<layer number="13" name="Route13" color="4" fill="5" visible="no" active="no"/>
+<layer number="14" name="Route14" color="1" fill="6" visible="no" active="no"/>
+<layer number="15" name="Route15" color="4" fill="6" visible="no" active="no"/>
+<layer number="16" name="Bottom" color="1" fill="1" visible="no" active="no"/>
+<layer number="17" name="Pads" color="2" fill="1" visible="no" active="no"/>
+<layer number="18" name="Vias" color="2" fill="1" visible="no" active="no"/>
+<layer number="19" name="Unrouted" color="6" fill="1" visible="no" active="no"/>
+<layer number="20" name="Dimension" color="15" fill="1" visible="no" active="no"/>
+<layer number="21" name="tPlace" color="7" fill="1" visible="no" active="no"/>
+<layer number="22" name="bPlace" color="7" fill="1" visible="no" active="no"/>
+<layer number="23" name="tOrigins" color="15" fill="1" visible="no" active="no"/>
+<layer number="24" name="bOrigins" color="15" fill="1" visible="no" active="no"/>
+<layer number="25" name="tNames" color="7" fill="1" visible="no" active="no"/>
+<layer number="26" name="bNames" color="7" fill="1" visible="no" active="no"/>
+<layer number="27" name="tValues" color="7" fill="1" visible="no" active="no"/>
+<layer number="28" name="bValues" color="7" fill="1" visible="no" active="no"/>
 <layer number="29" name="tStop" color="7" fill="3" visible="no" active="no"/>
 <layer number="30" name="bStop" color="7" fill="6" visible="no" active="no"/>
@@
 <layer number="35" name="tGlue" color="7" fill="4" visible="no" active="no"/>
 <layer number="36" name="bGlue" color="7" fill="5" visible="no" active="no"/>
-<layer number="37" name="tTest" color="7" fill="1" visible="yes" active="no"/>
-<layer number="38" name="bTest" color="7" fill="1" visible="yes" active="no"/>
+<layer number="37" name="tTest" color="7" fill="1" visible="no" active="no"/>
+<layer number="38" name="bTest" color="7" fill="1" visible="no" active="no"/>
 <layer number="39" name="tKeepout" color="4" fill="11" visible="no" active="no"/>
 <layer number="40" name="bKeepout" color="1" fill="11" visible="no" active="no"/>
@@
 <layer number="44" name="Drills" color="7" fill="1" visible="no" active="no"/>
 <layer number="45" name="Holes" color="7" fill="1" visible="no" active="no"/>
-<layer number="46" name="Milling" color="3" fill="1" visible="yes" active="no"/>
-<layer number="47" name="Measures" color="7" fill="1" visible="yes" active="no"/>
-<layer number="48" name="Document" color="7" fill="1" visible="yes" active="no"/>
-<layer number="49" name="Reference" color="7" fill="1" visible="yes" active="no"/>
-<layer number="50" name="dxf" color="7" fill="1" visible="yes" active="no"/>
-<layer number="51" name="tDocu" color="7" fill="1" visible="yes" active="no"/>
-<layer number="52" name="bDocu" color="7" fill="1" visible="yes" active="no"/>
-<layer number="53" name="tGND_GNDA" color="7" fill="9" visible="yes" active="no"/>
-<layer number="54" name="bGND_GNDA" color="1" fill="9" visible="yes" active="no"/>
-<layer number="56" name="wert" color="7" fill="1" visible="yes" active="no"/>
-<layer number="57" name="tCAD" color="7" fill="1" visible="yes" active="no"/>
-<layer number="59" name="tCarbon" color="7" fill="1" visible="yes" active="no"/>
-<layer number="60" name="bCarbon" color="7" fill="1" visible="yes" active="no"/>
+<layer number="46" name="Milling" color="3" fill="1" visible="no" active="no"/>
+<layer number="47" name="Measures" color="7" fill="1" visible="no" active="no"/>
+<layer number="48" name="Document" color="7" fill="1" visible="no" active="no"/>
+<layer number="49" name="Reference" color="7" fill="1" visible="no" active="no"/>
+<layer number="50" name="dxf" color="7" fill="1" visible="no" active="no"/>
+<layer number="51" name="tDocu" color="7" fill="1" visible="no" active="no"/>
+<layer number="52" name="bDocu" color="7" fill="1" visible="no" active="no"/>
+<layer number="53" name="tGND_GNDA" color="7" fill="9" visible="no" active="no"/>
+<layer number="54" name="bGND_GNDA" color="1" fill="9" visible="no" active="no"/>
+<layer number="56" name="wert" color="7" fill="1" visible="no" active="no"/>
+<layer number="57" name="tCAD" color="7" fill="1" visible="no" active="no"/>
+<layer number="59" name="tCarbon" color="7" fill="1" visible="no" active="no"/>
+<layer number="60" name="bCarbon" color="7" fill="1" visible="no" active="no"/>
 <layer number="88" name="SimResults" color="9" fill="1" visible="yes" active="yes"/>
 <layer number="89" name="SimProbes" color="9" fill="1" visible="yes" active="yes"/>
@@
 <part name="C10" library="rcl" library_urn="urn:adsk.eagle:library:334" deviceset="C-EU" device="C0603" value="10uF"/>
 <part name="C13" library="microbuilder" deviceset="CAP_TANTALUM" device="D/7343_REFLOW" value="100uF"/>
-<part name="P+6" library="supply1" library_urn="urn:adsk.eagle:library:371" deviceset="V+" device=""/>
+<part name="P+6" library="supply1" deviceset="+12V" device=""/>
 </parts>
 <sheets>
@@
 <instance part="C10" gate="G$1" x="381" y="266.7"/>
 <instance part="C13" gate="G$1" x="543.56" y="276.86"/>
-<instance part="P+6" gate="1" x="457.2" y="274.32"/>
+<instance part="P+6" gate="1" x="457.2" y="276.86"/>
 </instances>
 <busses>
@@
 <pinref part="C7" gate="G$1" pin="1"/>
 </segment>
+<segment>
+<pinref part="JP1" gate="G$1" pin="1"/>
+<wire x1="449.58" y1="248.92" x2="457.2" y2="248.92" width="0.1524" layer="91"/>
+<wire x1="457.2" y1="248.92" x2="457.2" y2="274.32" width="0.1524" layer="91"/>
+<pinref part="P+6" gate="1" pin="+12V"/>
+</segment>
 </net>
 <net name="N$4" class="0">
@@
 <junction x="25.4" y="299.72"/>
 </segment>
-<segment>
-<pinref part="JP1" gate="G$1" pin="1"/>
-<wire x1="449.58" y1="248.92" x2="457.2" y2="248.92" width="0.1524" layer="91"/>
-<wire x1="457.2" y1="248.92" x2="457.2" y2="271.78" width="0.1524" layer="91"/>
-<pinref part="P+6" gate="1" pin="V+"/>
-</segment>
-</net>
+</net>

Commit message: Add files via upload
Changes made to MEMS board V08
Parts:
- added C15: 10uF, rcl:C-EUC0603
- L1: device SparkFun-Passives:INDUCTOR0603 -> SparkFun-Passives:INDUCTORCR54
Connections:
- net GROU[ renamed N$21
- new net N$23: C15.2, R13.1
- new net VUSB: C1.1, IC2.VIN, J1.VBUS
- net +12V: no longer R11.2
- net N$1: now also R11.2
- net N$3: now also C15.1; no longer R13.1
- net V+: no longer C1.1, IC2.VIN, J1.VBUS
Changed lines of the file:
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@@
 <part name="GND15" library="supply1" deviceset="GND" device=""/>
 <part name="P+8" library="supply1" deviceset="+12V" device=""/>
-<part name="P+7" library="supply1" deviceset="+12V" device=""/>
 <part name="R15" library="CMU-ArtFab" deviceset="R-US_" device="R0603" value="1k"/>
 <part name="POT1" library="CMU-ArtFab" deviceset="POT-DUAL-PTV112" device="-4420" value="20K"/>
@@
 <part name="R3" library="CMU-ArtFab" deviceset="R-US_" device="R0603" value="1k"/>
 <part name="P+2" library="supply1" library_urn="urn:adsk.eagle:library:371" deviceset="V+" device=""/>
-<part name="P+1" library="supply1" library_urn="urn:adsk.eagle:library:371" deviceset="V+" device=""/>
 <part name="IC2" library="CMU-ArtFab" deviceset="BQ21040-LIPO-CHARGER" device="" value="BQ21040"/>
 <part name="R4" library="CMU-ArtFab" deviceset="R-US_" device="R0603" value="10k"/>
@@
 <part name="IC4" library="CMU-ArtFab" deviceset="SC4503" device=""/>
 <part name="J3" library="CMU-ArtFab" deviceset="TRS-1/8&quot;-3.5MM" device="" value=""/>
-<part name="L1" library="SparkFun-Passives" deviceset="INDUCTOR" device="0603" value="2.7uH"/>
+<part name="L1" library="SparkFun-Passives" deviceset="INDUCTOR" device="CR54" value="2.7uH"/>
 <part name="C6" library="rcl" library_urn="urn:adsk.eagle:library:334" deviceset="C-EU" device="C1206" value="68uF"/>
 <part name="C3" library="rcl" library_urn="urn:adsk.eagle:library:334" deviceset="C-EU" device="C0603" value="10uF"/>
@@
 <part name="C13" library="microbuilder" deviceset="CAP_TANTALUM" device="D/7343_REFLOW" value="100uF"/>
 <part name="P+6" library="supply1" deviceset="+12V" device=""/>
+<part name="P+1" library="supply1" library_urn="urn:adsk.eagle:library:371" deviceset="V+" device="" value="VUSB"/>
+<part name="C15" library="rcl" library_urn="urn:adsk.eagle:library:334" deviceset="C-EU" device="C0603" value="10uF"/>
 </parts>
 <sheets>
@@
 </instance>
 <instance part="P+8" gate="1" x="543.56" y="307.34"/>
-<instance part="P+7" gate="1" x="472.44" y="302.26"/>
 <instance part="R15" gate="G$1" x="553.72" y="259.08"/>
 <instance part="POT1" gate="/1" x="515.62" y="238.76" rot="R90"/>
@@
 <instance part="R3" gate="G$1" x="86.36" y="279.4" rot="R180"/>
 <instance part="P+2" gate="1" x="93.98" y="297.18"/>
-<instance part="P+1" gate="1" x="22.86" y="304.8"/>
 <instance part="IC2" gate="G$1" x="50.8" y="289.56" rot="MR0"/>
 <instance part="R4" gate="G$1" x="106.68" y="299.72" rot="R180"/>
@@
 <instance part="C13" gate="G$1" x="543.56" y="276.86"/>
 <instance part="P+6" gate="1" x="457.2" y="276.86"/>
+<instance part="P+1" gate="1" x="22.86" y="304.8"/>
+<instance part="C15" gate="G$1" x="462.28" y="256.54" rot="R90"/>
 </instances>
 <busses>
@@
 </segment>
 </net>
-<net name="N$3" class="0">
-<segment>
-<pinref part="JP1" gate="G$1" pin="4"/>
-<wire x1="449.58" y1="256.54" x2="472.44" y2="256.54" width="0.1524" layer="91"/>
-<pinref part="R13" gate="G$1" pin="1"/>
-</segment>
-</net>
 <net name="N$5" class="0">
 <segment>
@@
 <junction x="515.62" y="259.08"/>
 <pinref part="C12" gate="G$1" pin="1"/>
-</segment>
-</net>
-<net name="N$1" class="0">
-<segment>
-<pinref part="R14" gate="G$1" pin="1"/>
-<wire x1="543.56" y1="289.56" x2="543.56" y2="284.48" width="0.1524" layer="91"/>
-<pinref part="IC6" gate="A" pin="V+"/>
-<wire x1="543.56" y1="284.48" x2="543.56" y2="281.94" width="0.1524" layer="91"/>
-<wire x1="543.56" y1="284.48" x2="502.92" y2="284.48" width="0.1524" layer="91"/>
-<wire x1="502.92" y1="284.48" x2="502.92" y2="266.7" width="0.1524" layer="91"/>
-<junction x="543.56" y="284.48"/>
-<pinref part="C13" gate="G$1" pin="+"/>
 </segment>
 </net>
@@
 <wire x1="543.56" y1="304.8" x2="543.56" y2="299.72" width="0.1524" layer="91"/>
 <pinref part="P+8" gate="1" pin="+12V"/>
-</segment>
-<segment>
-<pinref part="R11" gate="G$1" pin="2"/>
-<wire x1="472.44" y1="299.72" x2="472.44" y2="297.18" width="0.1524" layer="91"/>
-<pinref part="P+7" gate="1" pin="+12V"/>
 </segment>
 <segment>
@@
 <junction x="591.82" y="259.08"/>
 <pinref part="C14" gate="G$1" pin="1"/>
-</segment>
-</net>
-<net name="GROU[" class="0">
-<segment>
-<pinref part="R15" gate="G$1" pin="2"/>
-<wire x1="558.8" y1="259.08" x2="563.88" y2="259.08" width="0.1524" layer="91"/>
-<wire x1="563.88" y1="259.08" x2="563.88" y2="256.54" width="0.1524" layer="91"/>
-<pinref part="IC6" gate="B" pin="-IN"/>
-<wire x1="563.88" y1="256.54" x2="568.96" y2="256.54" width="0.1524" layer="91"/>
-<wire x1="568.96" y1="256.54" x2="571.5" y2="256.54" width="0.1524" layer="91"/>
-<wire x1="584.2" y1="241.3" x2="568.96" y2="241.3" width="0.1524" layer="91"/>
-<wire x1="568.96" y1="241.3" x2="568.96" y2="256.54" width="0.1524" layer="91"/>
-<junction x="568.96" y="256.54"/>
-<pinref part="POT1" gate="/2" pin="E"/>
 </segment>
 </net>
@@
 <pinref part="P+2" gate="1" pin="V+"/>
 <wire x1="93.98" y1="294.64" x2="93.98" y2="292.1" width="0.1524" layer="91"/>
-</segment>
-<segment>
-<pinref part="P+1" gate="1" pin="V+"/>
-<wire x1="22.86" y1="302.26" x2="22.86" y2="299.72" width="0.1524" layer="91"/>
-<pinref part="J1" gate="G$1" pin="VBUS"/>
-<wire x1="22.86" y1="299.72" x2="17.78" y2="299.72" width="0.1524" layer="91"/>
-<pinref part="IC2" gate="G$1" pin="VIN"/>
-<wire x1="30.48" y1="299.72" x2="25.4" y2="299.72" width="0.1524" layer="91"/>
-<junction x="22.86" y="299.72"/>
-<pinref part="C1" gate="G$1" pin="1"/>
-<wire x1="25.4" y1="299.72" x2="22.86" y2="299.72" width="0.1524" layer="91"/>
-<junction x="25.4" y="299.72"/>
 </segment>
 </net>
@@
 </segment>
 </net>
+<net name="VUSB" class="0">
+<segment>
+<wire x1="22.86" y1="302.26" x2="22.86" y2="299.72" width="0.1524" layer="91"/>
+<pinref part="J1" gate="G$1" pin="VBUS"/>
+<wire x1="22.86" y1="299.72" x2="17.78" y2="299.72" width="0.1524" layer="91"/>
+<pinref part="IC2" gate="G$1" pin="VIN"/>
+<wire x1="30.48" y1="299.72" x2="25.4" y2="299.72" width="0.1524" layer="91"/>
+<junction x="22.86" y="299.72"/>
+<pinref part="C1" gate="G$1" pin="1"/>
+<wire x1="25.4" y1="299.72" x2="22.86" y2="299.72" width="0.1524" layer="91"/>
+<junction x="25.4" y="299.72"/>
+<pinref part="P+1" gate="1" pin="V+"/>
+</segment>
+</net>
+<net name="N$21" class="0">
+<segment>
+<pinref part="R15" gate="G$1" pin="2"/>
+<wire x1="558.8" y1="259.08" x2="568.96" y2="259.08" width="0.1524" layer="91"/>
+<wire x1="568.96" y1="259.08" x2="568.96" y2="256.54" width="0.1524" layer="91"/>
+<pinref part="IC6" gate="B" pin="-IN"/>
+<wire x1="568.96" y1="256.54" x2="571.5" y2="256.54" width="0.1524" layer="91"/>
+<pinref part="POT1" gate="/2" pin="E"/>
+<wire x1="568.96" y1="256.54" x2="568.96" y2="241.3" width="0.1524" layer="91"/>
+<wire x1="568.96" y1="241.3" x2="584.2" y2="241.3" width="0.1524" layer="91"/>
+<junction x="568.96" y="256.54"/>
+</segment>
+</net>
+<net name="N$3" class="0">
+<segment>
+<pinref part="JP1" gate="G$1" pin="4"/>
+<pinref part="C15" gate="G$1" pin="1"/>
+<wire x1="449.58" y1="256.54" x2="459.74" y2="256.54" width="0.1524" layer="91"/>
+</segment>
+</net>
+<net name="N$23" class="0">
+<segment>
+<pinref part="C15" gate="G$1" pin="2"/>
+<pinref part="R13" gate="G$1" pin="1"/>
+<wire x1="467.36" y1="256.54" x2="472.44" y2="256.54" width="0.1524" layer="91"/>
+</segment>
+</net>
+<net name="N$1" class="0">
+<segment>
+<pinref part="R11" gate="G$1" pin="2"/>
+<wire x1="472.44" y1="299.72" x2="472.44" y2="297.18" width="0.1524" layer="91"/>
+<pinref part="R14" gate="G$1" pin="1"/>
+<wire x1="543.56" y1="289.56" x2="543.56" y2="284.48" width="0.1524" layer="91"/>
+<pinref part="IC6" gate="A" pin="V+"/>
+<wire x1="543.56" y1="284.48" x2="543.56" y2="281.94" width="0.1524" layer="91"/>
+<wire x1="543.56" y1="284.48" x2="502.92" y2="284.48" width="0.1524" layer="91"/>
+<wire x1="502.92" y1="284.48" x2="502.92" y2="266.7" width="0.1524" layer="91"/>
+<junction x="543.56" y="284.48"/>
+<pinref part="C13" gate="G$1" pin="+"/>
+<wire x1="472.44" y1="299.72" x2="502.92" y2="299.72" width="0.1524" layer="91"/>
+<wire x1="502.92" y1="299.72" x2="502.92" y2="284.48" width="0.1524" layer="91"/>
+<junction x="502.92" y="284.48"/>
+</segment>
+</net>
 </nets>
 </sheet>
@@
 with this version.
 </note>
+<note version="8.3" severity="warning">
+Since Version 8.3, EAGLE supports URNs for individual library
+assets (packages, symbols, and devices). The URNs of those assets
+will not be understood (or retained) with this version.
+</note>
 </compatibility>

Commit message: Add files via upload
Parts:
- removed IC2: BQ21040, CMU-ArtFab:BQ21040-LIPO-CHARGER
- removed IC3: BQ297X, CMU-ArtFab:BQ297X-BATTERY-MANAGER
- removed J1: (no value), SparkFun-Connectors:USB_MICRO-BREDUCED_PASTE
- added C16: 4.7uF, rcl:C-EUC0603
- added J4: (no value), CMU-ArtFab:USB_MICRO-BREDUCED_PASTE
- added R22, R23: 10M, CMU-ArtFab:R-US_R0603
- added U$1: MCP73831, CMU-ArtFab:MCP73831
- added U$2: QS6K1, CMU-ArtFab:QS6K1
- C1: value 10uF -> 4.7uF
- IC1: value DMN2400 -> BQ297X; device CMU-ArtFab:DUAL-NFET-DMN2400 -> CMU-ArtFab:BQ297X-BATTERY-MANAGERLONG
- IC6: value OPA2134 -> TL072D; device linear:OPA2134UA -> linear:TL072D; IC_NAME OPA2134 -> (none)
- LED2: value (none) -> Charge
- R2: value 10k -> 470
- R3: value 1k -> 5k
- R4: value 10k -> 2.2k
- renumbered J2 to J5, R5 to R16, SW1 to SW3
Connections:
- removed net GND2: C1.2, C2.1, IC1.D1, IC2.GND, IC3.VSS, J1.GND, R2.1, R4.1, SW3.2
- removed net N$15: IC2.CHG, R3.2
- removed net N$16: IC2.TS, R4.2
- removed net N$17: IC2.CURRENT-SET, R2.2
- removed net N$18: C2.2, IC3.BAT, R16.2
- removed net N$19: IC1.D2, IC1.S1
- removed net N$20: IC1.G1, IC3.CHG-FET
- removed net VUSB: C1.1, IC2.VIN, J1.VBUS
- new net +5V: C1.1, J4.VBUS, LED2.A, U$1.4VDD
- new net BATGND: C2.1, IC1.VSS, SW3.2, U$2.6D1
- new net N$25: R2.2, U$1.1STAT
- new net N$27: IC1.DRAIN-FET, R23.2, U$2.1G1
- new net N$31: IC1.CHG-FET, R22.2, U$2.3G2
- new net N$34: IC1.V-, R4.2
- new net N$42: C2.2, IC1.BAT, R16.2
- new net USBGND: C1.2, C16.2, J4.GND, J5.2, R3.1, SW3.1, U$1.2VSS
- net GND: now also IC6P.V-, R22.1, R23.1, R4.1, U$2.2S2; no longer IC1.S2, IC3.V-, IC6A.V-
- net N$1: now also IC6P.V+; no longer IC6A.V+
- net N$10: now also IC6A.OUT; no longer IC6B.OUT
- net N$11: now also U$2.4D2, U$2.5S1; no longer LED2.C, R3.1
- net N$21: now also IC6A.-IN; no longer IC6B.-IN
- net N$22: now also LED2.C, R2.1; no longer IC1.G2, IC3.DRAIN-FET
- net N$5: now also IC6B.-IN; no longer IC6A.-IN
- net N$6: now also R3.2, U$1.5PROG; no longer J5.2, SW3.1
- net N$9: now also IC6B.OUT; no longer IC6A.OUT
- net V+: no longer LED2.A
- net VBAT: now also C16.1, U$1.3VBAT; no longer IC2.OUT
Other:
- note added: "I have searched for alternatives to the BQ2790 but it really is our best option even though its small."
- note added: "these 10M resistors are optional. only use them if the battery is not turning off"
- moved on the sheet: C2, IC6B, LED2, R2, R3, R4

Commit message: Add files via upload
Parts:
- removed C13: 100uF, microbuilder:CAP_TANTALUMD/7343_REFLOW
- removed IC6: TL072D, linear:TL072D
- removed R14: 10, CMU-ArtFab:R-US_R0603
- added C17: 0.1uF, adafruit:C-USC0805K
- added IC2: OPA2134UA, linear:OPA2134UA
- added L2: 100uH/500mA, rcl:L-EUL3225M
- C15: device rcl:C-EUC0603 -> rcl:C-EUC1206
Connections:
- removed net N$1: C13.+, IC6P.V+, R11.2, R14.1
- new net N$15: C17.1, IC2A.V+, L2.2, R11.2
- net +12V: now also L2.1; no longer R14.2
- net GND: now also C17.2, IC2A.V-; no longer C13.-, IC6P.V-
- net N$10: now also IC2B.OUT; no longer IC6A.OUT
- net N$21: now also IC2B.-IN; no longer IC6A.-IN
- net N$5: now also IC2A.-IN; no longer IC6B.-IN
- net N$8: now also IC2A.+IN, IC2B.+IN; no longer IC6A.+IN, IC6B.+IN
- net N$9: now also IC2A.OUT; no longer IC6B.OUT

Commit message: Add files via upload
IC names changed according to convention
Parts:
- renumbered U$1 to IC3, U$2 to IC6
