File: MEMS-preamp/MEMS-preamp_v08.sch (EAGLE design)
At the start: 49 parts, among them IC1 BQ297X, IC2 OPA2134UA, IC3 MCP73831, IC4 SC4503, IC5 TPS7A49, IC6 QS6K1, J3 TRS-1/8"-3.5MM, J5 Battery, SW3 SPDT

Commit message: MEMS preamp with electrolytic caps
Parts:
- removed C14: 10uF, adafruit:C-USC0805
- added C13: 10uF, resistor:CPOL-EUB
- C12: device adafruit:C-USC0805 -> resistor:CPOL-EUB
Connections:
- net N$10: now also C13.+; no longer C14.1
- net N$4: now also C12.-; no longer C12.2
- net N$7: now also C13.-; no longer C14.2
- net N$9: now also C12.+; no longer C12.1
Changed lines of the file:
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@@
 <?xml version="1.0" encoding="utf-8"?>
 <!DOCTYPE eagle SYSTEM "eagle.dtd">
-<eagle version="8.6.0">
+<eagle version="8.7.0">
 <drawing>
 <settings>
@@
 <part name="P+5" library="supply1" library_urn="urn:adsk.eagle:library:371" deviceset="V+" device=""/>
 <part name="C11" library="adafruit" deviceset="C-US" device="C0805" value="0.1uF"/>
-<part name="C14" library="adafruit" deviceset="C-US" device="C0805" value="10uF"/>
-<part name="C12" library="adafruit" library_urn="urn:adsk.eagle:library:420" deviceset="C-US" device="C0805" value="10uF"/>
 <part name="IC4" library="CMU-ArtFab" deviceset="SC4503" device=""/>
-<part name="J3" library="CMU-ArtFab" deviceset="TRS-1/8&quot;-3.5MM" device="" value=""/>
+<part name="J3" library="CMU-ArtFab" deviceset="TRS-1/8&quot;-3.5MM" device="" value="TRS-1/8&quot;-3.5MM"/>
 <part name="L1" library="SparkFun-Passives" deviceset="INDUCTOR" device="CR54" value="2.7uH"/>
 <part name="C6" library="rcl" library_urn="urn:adsk.eagle:library:334" deviceset="C-EU" device="C1206" package3d_urn="urn:adsk.eagle:package:23618/2" value="68uF"/>
@@
 <part name="L2" library="rcl" library_urn="urn:adsk.eagle:library:334" deviceset="L-EU" device="L3225M" package3d_urn="urn:adsk.eagle:package:23477/1" value="100uH/500mA"/>
 <part name="GND14" library="supply1" deviceset="GND" device=""/>
+<part name="C12" library="resistor" library_urn="urn:adsk.eagle:library:348" deviceset="CPOL-EU" device="B" package3d_urn="urn:adsk.eagle:package:25911/1" value="10uF"/>
+<part name="C13" library="resistor" library_urn="urn:adsk.eagle:library:348" deviceset="CPOL-EU" device="B" package3d_urn="urn:adsk.eagle:package:25911/1" value="10uF"/>
 </parts>
 <sheets>
@@
 <instance part="P+5" gate="1" x="370.84" y="287.02"/>
 <instance part="C11" gate="G$1" x="480.06" y="276.86"/>
-<instance part="C14" gate="G$1" x="599.44" y="259.08" rot="R90"/>
-<instance part="C12" gate="G$1" x="530.86" y="259.08" rot="R90"/>
 <instance part="IC4" gate="G$1" x="238.76" y="261.62" rot="MR0"/>
 <instance part="J3" gate="G$1" x="629.92" y="256.54" rot="R180"/>
@@
 <attribute name="VALUE" x="538.48" y="274.32" size="1.778" layer="96" ratio="12"/>
 </instance>
+<instance part="C12" gate="G$1" x="530.86" y="259.08" rot="R90"/>
+<instance part="C13" gate="G$1" x="599.44" y="259.08" rot="R90"/>
 </instances>
 <busses>
@@
 <wire x1="515.62" y1="243.84" x2="515.62" y2="259.08" width="0.1524" layer="91"/>
 <junction x="515.62" y="259.08"/>
-<pinref part="C12" gate="G$1" pin="1"/>
 <pinref part="IC2" gate="A" pin="OUT"/>
+<pinref part="C12" gate="G$1" pin="+"/>
 </segment>
 </net>
@@
 <wire x1="614.68" y1="256.54" x2="629.92" y2="256.54" width="0.1524" layer="91"/>
 <wire x1="604.52" y1="259.08" x2="614.68" y2="259.08" width="0.1524" layer="91"/>
-<pinref part="C14" gate="G$1" pin="2"/>
 <pinref part="J3" gate="G$1" pin="RING1"/>
 <pinref part="J3" gate="G$1" pin="TIP"/>
@@
 <wire x1="614.68" y1="261.62" x2="614.68" y2="259.08" width="0.1524" layer="91"/>
 <junction x="614.68" y="259.08"/>
+<pinref part="C13" gate="G$1" pin="-"/>
 </segment>
 </net>
@@
 <pinref part="R15" gate="G$1" pin="1"/>
 <wire x1="535.94" y1="259.08" x2="548.64" y2="259.08" width="0.1524" layer="91"/>
-<pinref part="C12" gate="G$1" pin="2"/>
+<pinref part="C12" gate="G$1" pin="-"/>
 </segment>
 </net>
@@
 <wire x1="591.82" y1="246.38" x2="591.82" y2="259.08" width="0.1524" layer="91"/>
 <junction x="591.82" y="259.08"/>
-<pinref part="C14" gate="G$1" pin="1"/>
 <pinref part="IC2" gate="B" pin="OUT"/>
-</segment>
-</net>
+<pinref part="C13" gate="G$1" pin="+"/>
+</segment>
+</net>

Commit message: MEMS preamp with electrolytic caps
Parts:
- removed C15: 10uF, rcl:C-EUC1206
- added C14: 10uF, resistor:CPOL-EUB
Connections:
- net N$23: now also C14.-; no longer C15.2
- net N$3: now also C14.+; no longer C15.1
Changed lines of the file:
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@@
 <part name="C10" library="rcl" library_urn="urn:adsk.eagle:library:334" deviceset="C-EU" device="C0603" package3d_urn="urn:adsk.eagle:package:23616/2" value="10uF"/>
 <part name="P+6" library="supply1" deviceset="+12V" device=""/>
-<part name="C15" library="rcl" library_urn="urn:adsk.eagle:library:334" deviceset="C-EU" device="C1206" package3d_urn="urn:adsk.eagle:package:23618/2" value="10uF"/>
 <part name="U4" library="microbuilder" deviceset="VBAT" device=""/>
 <part name="SW3" library="CMU-ArtFab" deviceset="SWITCH_SPDT" device="CL-SB-12B" value="SPDT"/>
@@
 <part name="C12" library="resistor" library_urn="urn:adsk.eagle:library:348" deviceset="CPOL-EU" device="B" package3d_urn="urn:adsk.eagle:package:25911/1" value="10uF"/>
 <part name="C13" library="resistor" library_urn="urn:adsk.eagle:library:348" deviceset="CPOL-EU" device="B" package3d_urn="urn:adsk.eagle:package:25911/1" value="10uF"/>
+<part name="C14" library="resistor" library_urn="urn:adsk.eagle:library:348" deviceset="CPOL-EU" device="B" package3d_urn="urn:adsk.eagle:package:25911/1" value="10uF"/>
 </parts>
 <sheets>
@@
 <instance part="C10" gate="G$1" x="381" y="266.7"/>
 <instance part="P+6" gate="1" x="457.2" y="276.86"/>
-<instance part="C15" gate="G$1" x="462.28" y="256.54" rot="R90"/>
 <instance part="U4" gate="G$1" x="154.94" y="302.26"/>
 <instance part="SW3" gate="G$1" x="162.56" y="287.02"/>
@@
 <instance part="C12" gate="G$1" x="530.86" y="259.08" rot="R90"/>
 <instance part="C13" gate="G$1" x="599.44" y="259.08" rot="R90"/>
+<instance part="C14" gate="G$1" x="462.28" y="256.54" rot="R90"/>
 </instances>
 <busses>
@@
 <segment>
 <pinref part="JP1" gate="G$1" pin="4"/>
-<pinref part="C15" gate="G$1" pin="1"/>
 <wire x1="449.58" y1="256.54" x2="459.74" y2="256.54" width="0.1524" layer="91"/>
+<pinref part="C14" gate="G$1" pin="+"/>
 </segment>
 </net>
 <net name="N$23" class="0">
 <segment>
-<pinref part="C15" gate="G$1" pin="2"/>
 <pinref part="R13" gate="G$1" pin="1"/>
 <wire x1="467.36" y1="256.54" x2="472.44" y2="256.54" width="0.1524" layer="91"/>
-</segment>
-</net>
+<pinref part="C14" gate="G$1" pin="-"/>
+</segment>
+</net>

Commit message: gerbers for mems and piezo
Parts:
- removed IC5: TPS7A49, CMU-ArtFab:TPS7A49
- removed R22, R23: 10M, CMU-ArtFab:R-US_R0603
- added R14: 150k, CMU-ArtFab:R-US_R0603
- added R5: 470, CMU-ArtFab:R-US_R0603
- added U3: MCP73831, CMU-ArtFab:MCP73831
- C10: value 10uF -> 10nF
- C11: value 0.1uF -> 10uF; device adafruit:C-USC0805 -> rcl:C-EUC0603
- C13: value 10uF -> 0.1uF; device resistor:CPOL-EUB -> adafruit:C-USC0805
- C16: value 4.7uF -> 10uF; device rcl:C-EUC0603 -> resistor:CPOL-EUB
- C2: value 0.1uF -> 4.7uF
- C3: value 10uF -> 0.1uF
- C4: value 56nF -> 10uF
- C5: value 2.2pF -> 56nF
- C6: value 68uF -> 2.2pF; device rcl:C-EUC1206 -> rcl:C-EUC0603
- C7: value 10uF -> 68uF; device rcl:C-EUC0603 -> rcl:C-EUC1206
- C8: value 10nF -> 10uF
- IC2: value OPA2134UA -> SC4503; device linear:OPA2134UA -> CMU-ArtFab:SC4503
- IC3: value MCP73831 -> TPS7A49; device CMU-ArtFab:MCP73831 -> CMU-ArtFab:TPS7A49
- IC4: value SC4503 -> OPA2134UA; device CMU-ArtFab:SC4503 -> linear:OPA2134UA
- R10: value 11k -> 100k
- R11: value 150k -> 100k
- R12: value 150k -> 11k
- R13: value 1k -> 150k
- R16: value 330 -> 1k
- R2: value 470 -> 5k
- R3: value 5k -> 10M
- R4: value 2.2k -> 10M
- R6: value 15k -> 2.2k
- R7: value 1M -> 330
- R8: value 100k -> 15k
- R9: value 100k -> 1M
- renumbered C17 to C15, IC6 to U2, J4 to J1, J5 to J2, SW3 to SW1
Connections:
- removed net N$23 (its old number): C14.-, R13.1
- new net N$4: C14.-, R16.1
- net +12V: now also C9.1, IC3.OUT, R11.1; no longer C7.1, IC5.OUT, R9.1
- net +5V: now also U3.4VDD; no longer IC3.4VDD
- net BATGND: now also C3.1; no longer C2.1
- net GND: now also C13.2, C5.2, C8.2, IC2.GND, IC3.GND, IC4A.V-, R10.1, R12.2, R14.1, R3.1, R6.1; no longer C3.2, C6.2, C9.2, IC2A.V-, IC4.GND, IC5.GND, R10.2, R12.1, R22.1, R23.1, R8.1
- net N$10: now also C16.+, IC4B.OUT; no longer C13.+, IC2B.OUT
- net N$12: now also IC2.SW; no longer IC4.SW
- net N$13: now also C5.1, IC2.SHDN, R8.1; no longer C4.1, IC4.SHDN, R6.1
- net N$14: now also C6.2, IC2.FB, R10.2, R9.1; no longer C5.2, IC4.FB, R7.1, R8.2
- net N$15: now also IC4A.V+, R13.2; no longer IC2A.V+, R11.2
- net N$21: now also IC4B.-IN, R16.2; no longer IC2B.-IN, R15.2
- net N$22: now also R5.1; no longer R2.1
- net N$25: now also R5.2, U3.1STAT; no longer IC3.1STAT, R2.2
- net N$27: now also R3.2; no longer R23.2
- net N$3: now also C12.+; no longer C14.+
- net N$31: now also R4.2; no longer R22.2
- net N$34: now also R6.2; no longer R4.2
- net N$42: now also C3.2, R7.2; no longer C2.2, R16.2
- net N$47: now also C9.2, IC3.FB, R11.2, R12.1; no longer C8.2, IC5.FB, R10.1, R9.2
- net N$48: now also C10.1, IC3.NR/SS; no longer C9.1, IC5.NR/SS
- net N$5: now also IC4A.-IN, R15.2; no longer IC2A.-IN, R13.2
- net N$6: now also R2.2, U3.5PROG; no longer IC3.5PROG, R3.2
- net N$7: now also C16.-; no longer C13.-
- net N$8: now also C13.1, IC4A.+IN, IC4B.+IN, R13.1, R14.2; no longer C11.1, IC2A.+IN, IC2B.+IN, R11.1, R12.2
- net N$9: now also C14.+, IC4A.OUT; no longer C12.+, IC2A.OUT
- net USBGND: now also C2.2, R2.1, U3.2VSS; no longer C16.2, IC3.2VSS, R3.1
- net V+: now also C11.1, C7.1, IC3.EN, IC3.IN, R9.2; no longer C10.1, C5.1, IC5.EN, IC5.IN, R7.2
- net VBAT: now also C2.1, C4.1, IC2.IN, R7.1, R8.2, U3.3VBAT; no longer C16.1, C3.1, IC3.3VBAT, IC4.IN, R16.1, R6.2
Other:
- moved on the sheet: C10, C11, C12, C14, C2, C3, C4, C5, C6, C7, C8, C9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
