File: MEMS-preamp/MEMS-preamp_v10.sch (EAGLE design)
At the start: 49 parts, among them IC1 BQ297X, IC2 SC4503, IC3 TPS7A49, IC4 OPA2134UA, J2 Battery, J3 TRS-1/8"-3.5MM, SW1 SPDT, U2 QS6K1, U3 MCP73831

Commit message: mems v10, rebuilt from v8, to have electrolytic caps
Parts:
- C12: device rcl:C-EUC1206 -> resistor:CPOL-EUB
- C14, C16: device adafruit:C-USC0805 -> resistor:CPOL-EUB
- D1: value B130-13-F -> 10BQ015
Connections:
- net N$10: now also C16.+; no longer C16.1
- net N$23: now also C12.-; no longer C12.2
- net N$3: now also C12.+; no longer C12.1
- net N$4: now also C14.-; no longer C14.2
- net N$7: now also C16.-; no longer C16.2
- net N$9: now also C14.+; no longer C14.1
Changed lines of the file:
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@@
 <part name="U1" library="microbuilder" deviceset="VBAT" device=""/>
 <part name="U7" library="microbuilder" deviceset="VBAT" device=""/>
-<part name="D1" library="SparkFun" deviceset="DIODE" device="SMA" value="B130-13-F"/>
+<part name="D1" library="SparkFun" deviceset="DIODE" device="SMA" value="10BQ015"/>
 <part name="GND4" library="SparkFun" deviceset="GND" device=""/>
 <part name="GND8" library="SparkFun" deviceset="GND" device=""/>
@@
 <part name="P+5" library="supply1" library_urn="urn:adsk.eagle:library:371" deviceset="V+" device=""/>
 <part name="C13" library="adafruit" deviceset="C-US" device="C0805" value="0.1uF"/>
-<part name="C16" library="adafruit" deviceset="C-US" device="C0805" value="10uF"/>
-<part name="C14" library="adafruit" library_urn="urn:adsk.eagle:library:420" deviceset="C-US" device="C0805" value="10uF"/>
 <part name="IC2" library="CMU-ArtFab" deviceset="SC4503" device=""/>
 <part name="J3" library="CMU-ArtFab" deviceset="TRS-1/8&quot;-3.5MM" device="" value="TRS-1/8&quot;-3.5MM"/>
@@
 <part name="C11" library="rcl" library_urn="urn:adsk.eagle:library:334" deviceset="C-EU" device="C0603" package3d_urn="urn:adsk.eagle:package:23616/2" value="10uF"/>
 <part name="P+6" library="supply1" deviceset="+12V" device=""/>
-<part name="C12" library="rcl" library_urn="urn:adsk.eagle:library:334" deviceset="C-EU" device="C1206" package3d_urn="urn:adsk.eagle:package:23618/2" value="10uF"/>
 <part name="U6" library="microbuilder" deviceset="VBAT" device=""/>
 <part name="SW1" library="CMU-ArtFab" deviceset="SWITCH_SPDT" device="CL-SB-12B" value="SPDT"/>
@@
 <part name="L2" library="rcl" library_urn="urn:adsk.eagle:library:334" deviceset="L-EU" device="L3225M" package3d_urn="urn:adsk.eagle:package:23477/1" value="100uH/500mA"/>
 <part name="GND14" library="supply1" deviceset="GND" device=""/>
+<part name="C14" library="resistor" library_urn="urn:adsk.eagle:library:348" deviceset="CPOL-EU" device="B" package3d_urn="urn:adsk.eagle:package:25911/1" value="10uF"/>
+<part name="C16" library="resistor" library_urn="urn:adsk.eagle:library:348" deviceset="CPOL-EU" device="B" package3d_urn="urn:adsk.eagle:package:25911/1" value="10uF"/>
+<part name="C12" library="resistor" library_urn="urn:adsk.eagle:library:348" deviceset="CPOL-EU" device="B" package3d_urn="urn:adsk.eagle:package:25911/1" value="10uF"/>
 </parts>
 <sheets>
@@
 <instance part="P+5" gate="1" x="370.84" y="287.02"/>
 <instance part="C13" gate="G$1" x="480.06" y="276.86"/>
-<instance part="C16" gate="G$1" x="599.44" y="259.08" rot="R90"/>
-<instance part="C14" gate="G$1" x="530.86" y="259.08" rot="R90"/>
 <instance part="IC2" gate="G$1" x="238.76" y="261.62" rot="MR0"/>
 <instance part="J3" gate="G$1" x="629.92" y="256.54" rot="R180"/>
@@
 <instance part="C11" gate="G$1" x="381" y="266.7"/>
 <instance part="P+6" gate="1" x="457.2" y="276.86"/>
-<instance part="C12" gate="G$1" x="462.28" y="256.54" rot="R90"/>
 <instance part="U6" gate="G$1" x="154.94" y="302.26"/>
 <instance part="SW1" gate="G$1" x="162.56" y="287.02"/>
@@
 <attribute name="VALUE" x="538.48" y="274.32" size="1.778" layer="96" ratio="12"/>
 </instance>
+<instance part="C14" gate="G$1" x="530.86" y="259.08" rot="R90"/>
+<instance part="C16" gate="G$1" x="599.44" y="259.08" rot="R90"/>
+<instance part="C12" gate="G$1" x="462.28" y="256.54" rot="R90"/>
 </instances>
 <busses>
@@
 <wire x1="515.62" y1="243.84" x2="515.62" y2="259.08" width="0.1524" layer="91"/>
 <junction x="515.62" y="259.08"/>
-<pinref part="C14" gate="G$1" pin="1"/>
 <pinref part="IC4" gate="A" pin="OUT"/>
+<pinref part="C14" gate="G$1" pin="+"/>
 </segment>
 </net>
@@
 <wire x1="614.68" y1="256.54" x2="629.92" y2="256.54" width="0.1524" layer="91"/>
 <wire x1="604.52" y1="259.08" x2="614.68" y2="259.08" width="0.1524" layer="91"/>
-<pinref part="C16" gate="G$1" pin="2"/>
 <pinref part="J3" gate="G$1" pin="RING1"/>
 <pinref part="J3" gate="G$1" pin="TIP"/>
@@
 <wire x1="614.68" y1="261.62" x2="614.68" y2="259.08" width="0.1524" layer="91"/>
 <junction x="614.68" y="259.08"/>
+<pinref part="C16" gate="G$1" pin="-"/>
 </segment>
 </net>
@@
 <pinref part="R16" gate="G$1" pin="1"/>
 <wire x1="535.94" y1="259.08" x2="548.64" y2="259.08" width="0.1524" layer="91"/>
-<pinref part="C14" gate="G$1" pin="2"/>
+<pinref part="C14" gate="G$1" pin="-"/>
 </segment>
 </net>
@@
 <wire x1="591.82" y1="246.38" x2="591.82" y2="259.08" width="0.1524" layer="91"/>
 <junction x="591.82" y="259.08"/>
-<pinref part="C16" gate="G$1" pin="1"/>
 <pinref part="IC4" gate="B" pin="OUT"/>
+<pinref part="C16" gate="G$1" pin="+"/>
 </segment>
 </net>
@@
 <segment>
 <pinref part="JP1" gate="G$1" pin="4"/>
-<pinref part="C12" gate="G$1" pin="1"/>
 <wire x1="449.58" y1="256.54" x2="459.74" y2="256.54" width="0.1524" layer="91"/>
+<pinref part="C12" gate="G$1" pin="+"/>
 </segment>
 </net>
 <net name="N$23" class="0">
 <segment>
-<pinref part="C12" gate="G$1" pin="2"/>
 <pinref part="R15" gate="G$1" pin="1"/>
 <wire x1="467.36" y1="256.54" x2="472.44" y2="256.54" width="0.1524" layer="91"/>
-</segment>
-</net>
+<pinref part="C12" gate="G$1" pin="-"/>
+</segment>
+</net>

Commit message: mems v10, rebuilt from v8, to have electrolytic caps
Parts:
- D1: value 10BQ015 -> B130-13-F
Changed lines of the file:
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@@
 <part name="U1" library="microbuilder" deviceset="VBAT" device=""/>
 <part name="U7" library="microbuilder" deviceset="VBAT" device=""/>
-<part name="D1" library="SparkFun" deviceset="DIODE" device="SMA" value="10BQ015"/>
+<part name="D1" library="SparkFun" deviceset="DIODE" device="SMA" value="B130-13-F"/>
 <part name="GND4" library="SparkFun" deviceset="GND" device=""/>
 <part name="GND8" library="SparkFun" deviceset="GND" device=""/>

Commit message: v10 board updated to solve inconsistencies.
v08 local copy board was taken as reference and all the updates later were added in order to get a consistent board.
Parts:
- removed U3: MCP73831, CMU-ArtFab:MCP73831
- added IC5: TPS7A49, CMU-ArtFab:TPS7A49
- C12: value 10uF -> 0.1uF; device resistor:CPOL-EUB -> adafruit:C-USC0805
- C13: value 0.1uF -> 10uF; device adafruit:C-USC0805 -> rcl:C-EUC1206
- C14: value 10uF -> 0.1uF; device resistor:CPOL-EUB -> adafruit:C-USC0805K
- C15: value 0.1uF -> 10uF; device adafruit:C-USC0805K -> adafruit:C-USC0805
- C16: device resistor:CPOL-EUB -> adafruit:C-USC0805
- D1: value B130-13-F -> B-130-13-F
- IC2: value SC4503 -> OPA2134UA; device CMU-ArtFab:SC4503 -> linear:OPA2134UA
- IC3: value TPS7A49 -> MCP73831; device CMU-ArtFab:TPS7A49 -> CMU-ArtFab:MCP73831
- IC4: value OPA2134UA -> SC4503; device linear:OPA2134UA -> CMU-ArtFab:SC4503
- POT1: value 20K -> 10K
- R2: value 4.7K -> 470
- R3: value 10M -> 4.7k
- R5: value 470 -> 10M
- renumbered J1 to J4, J2 to J5, SW1 to SW3, U2 to IC6
Connections:
- net +12V: now also IC5.OUT; no longer IC3.OUT
- net +5V: now also IC3.4VDD; no longer U3.4VDD
- net GND: now also C12.2, C14.2, IC2A.V-, IC4.GND, IC5.GND, R5.1; no longer C13.2, C15.2, IC2.GND, IC3.GND, IC4A.V-, R3.1
- net N$10: now also C16.1, IC2B.OUT; no longer C16.+, IC4B.OUT
- net N$12: now also IC4.SW; no longer IC2.SW
- net N$13: now also IC4.SHDN; no longer IC2.SHDN
- net N$14: now also IC4.FB; no longer IC2.FB
- net N$15: now also C14.1, IC2A.V+; no longer C15.1, IC4A.V+
- net N$21: now also IC2B.-IN; no longer IC4B.-IN
- net N$22: now also R2.1; no longer R5.1
- net N$23: now also C13.2; no longer C12.-
- net N$25: now also IC3.1STAT, R2.2; no longer R5.2, U3.1STAT
- net N$27: now also R4.2; no longer R3.2
- net N$3: now also C13.1; no longer C12.+
- net N$31: now also R5.2; no longer R4.2
- net N$4: now also C15.2; no longer C14.-
- net N$47: now also IC5.FB; no longer IC3.FB
- net N$48: now also IC5.NR/SS; no longer IC3.NR/SS
- net N$5: now also IC2A.-IN; no longer IC4A.-IN
- net N$6: now also IC3.5PROG, R3.2; no longer R2.2, U3.5PROG
- net N$7: now also C16.2; no longer C16.-
- net N$8: now also C12.1, IC2A.+IN, IC2B.+IN; no longer C13.1, IC4A.+IN, IC4B.+IN
- net N$9: now also C15.1, IC2A.OUT; no longer C14.+, IC4A.OUT
- net USBGND: now also IC3.2VSS, R3.1; no longer R2.1, U3.2VSS
- net V+: now also IC5.EN, IC5.IN; no longer IC3.EN, IC3.IN
- net VBAT: now also IC3.3VBAT, IC4.IN; no longer IC2.IN, U3.3VBAT
Other:
- moved on the sheet: C13, C15, R2, R3, R4, R5

Commit message: Capacitors changed according to V08
Parts:
- C13: device rcl:C-EUC1206 -> resistor:CPOL-EUB
- C15, C16: device adafruit:C-USC0805 -> resistor:CPOL-EUB
Connections:
- net N$10: now also C16.+; no longer C16.1
- net N$23: now also C13.-; no longer C13.2
- net N$3: now also C13.+; no longer C13.1
- net N$4: now also C15.-; no longer C15.2
- net N$7: now also C16.-; no longer C16.2
- net N$9: now also C15.+; no longer C15.1
Changed lines of the file:
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@@
 <part name="P+5" library="supply1" library_urn="urn:adsk.eagle:library:371" deviceset="V+" device=""/>
 <part name="C12" library="adafruit" deviceset="C-US" device="C0805" value="0.1uF"/>
-<part name="C16" library="adafruit" deviceset="C-US" device="C0805" value="10uF"/>
-<part name="C15" library="adafruit" library_urn="urn:adsk.eagle:library:420" deviceset="C-US" device="C0805" value="10uF"/>
+<part name="C16" library="resistor" library_urn="urn:adsk.eagle:library:348" deviceset="CPOL-EU" device="B" package3d_urn="urn:adsk.eagle:package:25911/1" value="10uF"/>
+<part name="C15" library="resistor" library_urn="urn:adsk.eagle:library:348" deviceset="CPOL-EU" device="B" package3d_urn="urn:adsk.eagle:package:25911/1" value="10uF"/>
 <part name="IC4" library="CMU-ArtFab" deviceset="SC4503" device=""/>
 <part name="J3" library="CMU-ArtFab" deviceset="TRS-1/8&quot;-3.5MM" device="" value=""/>
@@
 <part name="C11" library="rcl" library_urn="urn:adsk.eagle:library:334" deviceset="C-EU" device="C0603" package3d_urn="urn:adsk.eagle:package:23616/2" value="10uF"/>
 <part name="P+6" library="supply1" deviceset="+12V" device=""/>
-<part name="C13" library="rcl" library_urn="urn:adsk.eagle:library:334" deviceset="C-EU" device="C1206" package3d_urn="urn:adsk.eagle:package:23618/2" value="10uF"/>
+<part name="C13" library="resistor" library_urn="urn:adsk.eagle:library:348" deviceset="CPOL-EU" device="B" package3d_urn="urn:adsk.eagle:package:25911/1" value="10uF"/>
 <part name="U4" library="microbuilder" deviceset="VBAT" device=""/>
 <part name="SW3" library="CMU-ArtFab" deviceset="SWITCH_SPDT" device="CL-SB-12B" value="SPDT"/>
@@
 <wire x1="515.62" y1="243.84" x2="515.62" y2="259.08" width="0.1524" layer="91"/>
 <junction x="515.62" y="259.08"/>
-<pinref part="C15" gate="G$1" pin="1"/>
+<pinref part="C15" gate="G$1" pin="+"/>
 <pinref part="IC2" gate="A" pin="OUT"/>
 </segment>
@@
 <wire x1="614.68" y1="256.54" x2="629.92" y2="256.54" width="0.1524" layer="91"/>
 <wire x1="604.52" y1="259.08" x2="614.68" y2="259.08" width="0.1524" layer="91"/>
-<pinref part="C16" gate="G$1" pin="2"/>
+<pinref part="C16" gate="G$1" pin="-"/>
 <pinref part="J3" gate="G$1" pin="RING1"/>
 <pinref part="J3" gate="G$1" pin="TIP"/>
@@
 <pinref part="R16" gate="G$1" pin="1"/>
 <wire x1="535.94" y1="259.08" x2="548.64" y2="259.08" width="0.1524" layer="91"/>
-<pinref part="C15" gate="G$1" pin="2"/>
+<pinref part="C15" gate="G$1" pin="-"/>
 </segment>
 </net>
@@
 <wire x1="591.82" y1="246.38" x2="591.82" y2="259.08" width="0.1524" layer="91"/>
 <junction x="591.82" y="259.08"/>
-<pinref part="C16" gate="G$1" pin="1"/>
+<pinref part="C16" gate="G$1" pin="+"/>
 <pinref part="IC2" gate="B" pin="OUT"/>
 </segment>
@@
 <segment>
 <pinref part="JP1" gate="G$1" pin="4"/>
-<pinref part="C13" gate="G$1" pin="1"/>
+<pinref part="C13" gate="G$1" pin="+"/>
 <wire x1="449.58" y1="256.54" x2="459.74" y2="256.54" width="0.1524" layer="91"/>
 </segment>
@@
 <net name="N$23" class="0">
 <segment>
-<pinref part="C13" gate="G$1" pin="2"/>
+<pinref part="C13" gate="G$1" pin="-"/>
 <pinref part="R15" gate="G$1" pin="1"/>
 <wire x1="467.36" y1="256.54" x2="472.44" y2="256.54" width="0.1524" layer="91"/>

Commit message: MEMS brd updated for C13, C15 and C16 layer issues
Parts:
- C13, C15, C16: device resistor:CPOL-EUB -> CMU-ArtFab:CPOL-EUB
Changed lines of the file:
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@@
 <grid distance="0.1" unitdist="inch" unit="inch" style="lines" multiple="1" display="no" altdistance="0.01" altunitdist="inch" altunit="inch"/>
 <layers>
-<layer number="1" name="Top" color="4" fill="1" visible="no" active="no"/>
-<layer number="2" name="Route2" color="1" fill="3" visible="no" active="no"/>
-<layer number="3" name="Route3" color="4" fill="3" visible="no" active="no"/>
-<layer number="4" name="Route4" color="1" fill="4" visible="no" active="no"/>
-<layer number="5" name="Route5" color="4" fill="4" visible="no" active="no"/>
-<layer number="6" name="Route6" color="1" fill="8" visible="no" active="no"/>
-<layer number="7" name="Route7" color="4" fill="8" visible="no" active="no"/>
-<layer number="8" name="Route8" color="1" fill="2" visible="no" active="no"/>
-<layer number="9" name="Route9" color="4" fill="2" visible="no" active="no"/>
-<layer number="10" name="Route10" color="1" fill="7" visible="no" active="no"/>
-<layer number="11" name="Route11" color="4" fill="7" visible="no" active="no"/>
-<layer number="12" name="Route12" color="1" fill="5" visible="no" active="no"/>
-<layer number="13" name="Route13" color="4" fill="5" visible="no" active="no"/>
-<layer number="14" name="Route14" color="1" fill="6" visible="no" active="no"/>
-<layer number="15" name="Route15" color="4" fill="6" visible="no" active="no"/>
-<layer number="16" name="Bottom" color="1" fill="1" visible="no" active="no"/>
-<layer number="17" name="Pads" color="2" fill="1" visible="no" active="no"/>
-<layer number="18" name="Vias" color="2" fill="1" visible="no" active="no"/>
-<layer number="19" name="Unrouted" color="6" fill="1" visible="no" active="no"/>
-<layer number="20" name="Dimension" color="15" fill="1" visible="no" active="no"/>
-<layer number="21" name="tPlace" color="7" fill="1" visible="no" active="no"/>
-<layer number="22" name="bPlace" color="7" fill="1" visible="no" active="no"/>
-<layer number="23" name="tOrigins" color="15" fill="1" visible="no" active="no"/>
-<layer number="24" name="bOrigins" color="15" fill="1" visible="no" active="no"/>
-<layer number="25" name="tNames" color="7" fill="1" visible="no" active="no"/>
-<layer number="26" name="bNames" color="7" fill="1" visible="no" active="no"/>
-<layer number="27" name="tValues" color="7" fill="1" visible="no" active="no"/>
-<layer number="28" name="bValues" color="7" fill="1" visible="no" active="no"/>
+<layer number="1" name="Top" color="4" fill="1" visible="yes" active="no"/>
+<layer number="2" name="Route2" color="1" fill="3" visible="yes" active="no"/>
+<layer number="3" name="Route3" color="4" fill="3" visible="yes" active="no"/>
+<layer number="4" name="Route4" color="1" fill="4" visible="yes" active="no"/>
+<layer number="5" name="Route5" color="4" fill="4" visible="yes" active="no"/>
+<layer number="6" name="Route6" color="1" fill="8" visible="yes" active="no"/>
+<layer number="7" name="Route7" color="4" fill="8" visible="yes" active="no"/>
+<layer number="8" name="Route8" color="1" fill="2" visible="yes" active="no"/>
+<layer number="9" name="Route9" color="4" fill="2" visible="yes" active="no"/>
+<layer number="10" name="Route10" color="1" fill="7" visible="yes" active="no"/>
+<layer number="11" name="Route11" color="4" fill="7" visible="yes" active="no"/>
+<layer number="12" name="Route12" color="1" fill="5" visible="yes" active="no"/>
+<layer number="13" name="Route13" color="4" fill="5" visible="yes" active="no"/>
+<layer number="14" name="Route14" color="1" fill="6" visible="yes" active="no"/>
+<layer number="15" name="Route15" color="4" fill="6" visible="yes" active="no"/>
+<layer number="16" name="Bottom" color="1" fill="1" visible="yes" active="no"/>
+<layer number="17" name="Pads" color="2" fill="1" visible="yes" active="no"/>
+<layer number="18" name="Vias" color="2" fill="1" visible="yes" active="no"/>
+<layer number="19" name="Unrouted" color="6" fill="1" visible="yes" active="no"/>
+<layer number="20" name="Dimension" color="15" fill="1" visible="yes" active="no"/>
+<layer number="21" name="tPlace" color="7" fill="1" visible="yes" active="no"/>
+<layer number="22" name="bPlace" color="7" fill="1" visible="yes" active="no"/>
+<layer number="23" name="tOrigins" color="15" fill="1" visible="yes" active="no"/>
+<layer number="24" name="bOrigins" color="15" fill="1" visible="yes" active="no"/>
+<layer number="25" name="tNames" color="7" fill="1" visible="yes" active="no"/>
+<layer number="26" name="bNames" color="7" fill="1" visible="yes" active="no"/>
+<layer number="27" name="tValues" color="7" fill="1" visible="yes" active="no"/>
+<layer number="28" name="bValues" color="7" fill="1" visible="yes" active="no"/>
 <layer number="29" name="tStop" color="7" fill="3" visible="no" active="no"/>
 <layer number="30" name="bStop" color="7" fill="6" visible="no" active="no"/>
@@
 <layer number="35" name="tGlue" color="7" fill="4" visible="no" active="no"/>
 <layer number="36" name="bGlue" color="7" fill="5" visible="no" active="no"/>
-<layer number="37" name="tTest" color="7" fill="1" visible="no" active="no"/>
-<layer number="38" name="bTest" color="7" fill="1" visible="no" active="no"/>
+<layer number="37" name="tTest" color="7" fill="1" visible="yes" active="no"/>
+<layer number="38" name="bTest" color="7" fill="1" visible="yes" active="no"/>
 <layer number="39" name="tKeepout" color="4" fill="11" visible="no" active="no"/>
 <layer number="40" name="bKeepout" color="1" fill="11" visible="no" active="no"/>
@@
 <layer number="44" name="Drills" color="7" fill="1" visible="no" active="no"/>
 <layer number="45" name="Holes" color="7" fill="1" visible="no" active="no"/>
-<layer number="46" name="Milling" color="3" fill="1" visible="no" active="no"/>
-<layer number="47" name="Measures" color="7" fill="1" visible="no" active="no"/>
-<layer number="48" name="Document" color="7" fill="1" visible="no" active="no"/>
-<layer number="49" name="Reference" color="7" fill="1" visible="no" active="no"/>
-<layer number="50" name="dxf" color="7" fill="1" visible="no" active="no"/>
-<layer number="51" name="tDocu" color="7" fill="1" visible="no" active="no"/>
-<layer number="52" name="bDocu" color="7" fill="1" visible="no" active="no"/>
-<layer number="53" name="tGND_GNDA" color="7" fill="9" visible="no" active="no"/>
-<layer number="54" name="bGND_GNDA" color="1" fill="9" visible="no" active="no"/>
-<layer number="56" name="wert" color="7" fill="1" visible="no" active="no"/>
-<layer number="57" name="tCAD" color="7" fill="1" visible="no" active="no"/>
-<layer number="59" name="tCarbon" color="7" fill="1" visible="no" active="no"/>
-<layer number="60" name="bCarbon" color="7" fill="1" visible="no" active="no"/>
+<layer number="46" name="Milling" color="3" fill="1" visible="yes" active="no"/>
+<layer number="47" name="Measures" color="7" fill="1" visible="yes" active="no"/>
+<layer number="48" name="Document" color="7" fill="1" visible="yes" active="no"/>
+<layer number="49" name="Reference" color="7" fill="1" visible="yes" active="no"/>
+<layer number="50" name="dxf" color="7" fill="1" visible="yes" active="no"/>
+<layer number="51" name="tDocu" color="7" fill="1" visible="yes" active="no"/>
+<layer number="52" name="bDocu" color="7" fill="1" visible="yes" active="no"/>
+<layer number="53" name="tGND_GNDA" color="7" fill="9" visible="yes" active="no"/>
+<layer number="54" name="bGND_GNDA" color="1" fill="9" visible="yes" active="no"/>
+<layer number="56" name="wert" color="7" fill="1" visible="yes" active="no"/>
+<layer number="57" name="tCAD" color="7" fill="1" visible="yes" active="no"/>
+<layer number="59" name="tCarbon" color="7" fill="1" visible="yes" active="no"/>
+<layer number="60" name="bCarbon" color="7" fill="1" visible="yes" active="no"/>
 <layer number="88" name="SimResults" color="9" fill="1" visible="yes" active="yes"/>
 <layer number="89" name="SimProbes" color="9" fill="1" visible="yes" active="yes"/>
@@
 <part name="P+5" library="supply1" library_urn="urn:adsk.eagle:library:371" deviceset="V+" device=""/>
 <part name="C12" library="adafruit" deviceset="C-US" device="C0805" value="0.1uF"/>
-<part name="C16" library="resistor" library_urn="urn:adsk.eagle:library:348" deviceset="CPOL-EU" device="B" package3d_urn="urn:adsk.eagle:package:25911/1" value="10uF"/>
-<part name="C15" library="resistor" library_urn="urn:adsk.eagle:library:348" deviceset="CPOL-EU" device="B" package3d_urn="urn:adsk.eagle:package:25911/1" value="10uF"/>
+<part name="C16" library="CMU-ArtFab" deviceset="CPOL-EU" device="B" value="10uF"/>
+<part name="C15" library="CMU-ArtFab" deviceset="CPOL-EU" device="B" value="10uF"/>
 <part name="IC4" library="CMU-ArtFab" deviceset="SC4503" device=""/>
 <part name="J3" library="CMU-ArtFab" deviceset="TRS-1/8&quot;-3.5MM" device="" value=""/>
@@
 <part name="C11" library="rcl" library_urn="urn:adsk.eagle:library:334" deviceset="C-EU" device="C0603" package3d_urn="urn:adsk.eagle:package:23616/2" value="10uF"/>
 <part name="P+6" library="supply1" deviceset="+12V" device=""/>
-<part name="C13" library="resistor" library_urn="urn:adsk.eagle:library:348" deviceset="CPOL-EU" device="B" package3d_urn="urn:adsk.eagle:package:25911/1" value="10uF"/>
+<part name="C13" library="CMU-ArtFab" deviceset="CPOL-EU" device="B" value="10uF"/>
 <part name="U4" library="microbuilder" deviceset="VBAT" device=""/>
 <part name="SW3" library="CMU-ArtFab" deviceset="SWITCH_SPDT" device="CL-SB-12B" value="SPDT"/>
