File: MEMS-preamp/MEMS-preamp_v13b_VBAT.brd (EAGLE design)
At the start: 100 x 20 mm, 49 parts, among them IC10 MCP73831, IC11 QS6K1, IC2 OPA2134UA, IC7 TPS7A49, IC8 BQ297X, IC9 SC4503, J1 Battery, SW1 SPDT

Commit message: rev14
Parts:
- moved R15 12.2 mm to (-38.6, -8.41)
- moved C15 9.37 mm to (-48.6, -15.3), turned to 0 degrees
- moved C16 6.80 mm to (-55.6, -15.4), turned to 0 degrees
- moved C14 4.00 mm to (-37.6, -2.70)
- moved R16 2.53 mm to (-40.3, -16.1)
- moved C12 1.61 mm to (-44.1, -12.4)
- moved R13 0.81 mm to (-43.9, -2.76)
- moved R14 0.70 mm to (-50.1, -2.81)
- moved C13 0.14 mm to (-49.4, -8.60)
Connections:
- net +12V: no longer JP1.1
- net VBAT: now also JP1.1
Routing:
- net GND: track 0.00 -> 256.7 mm, vias 0 -> 5
- net VBAT: track 0.00 -> 122.1 mm, vias 0 -> 3
- net +12V: track 0.00 -> 104.1 mm, vias 0 -> 4
- net V+: track 0.00 -> 77.7 mm, vias 0 -> 3
- net N$13: track 0.00 -> 70.8 mm, vias 0 -> 4
- net N$16: track 0.00 -> 55.1 mm, vias 0 -> 2
- net USBGND1: track 0.00 -> 53.8 mm, vias 0 -> 2
- net BATGND1: track 0.00 -> 48.4 mm, vias 0 -> 3
- net +5V: track 0.00 -> 48.4 mm, vias 0 -> 2
- net N$9: track 0.00 -> 47.0 mm, vias 0 -> 1
- net N$12: track 0.00 -> 45.7 mm, vias 0 -> 3
- net N$10: track 0.00 -> 42.7 mm
- net N$19: track 0.00 -> 39.4 mm
- net N$6: track 0.00 -> 38.5 mm, vias 0 -> 1
- net N$14: track 0.00 -> 38.4 mm, vias 0 -> 2
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Other:
- board text added: "MEMS-rev-13b"
- board text removed: "MEMS-rev-13"
