File: Chipchestra/chipchestra-v05-buttons.sch (EAGLE design)
At the start: 32 parts, among them U2 MCP23017SS

Commit message: new tickler boards, new chipchestra boards
Parts:
- LED: value VCC -> (none)
- renumbered BUTTON0 to B0, BUTTON1 to B1, BUTTON10 to B11, BUTTON11 to B10, BUTTON12 to B13, BUTTON13 to B12, BUTTON14 to B15, BUTTON15 to B14, BUTTON2 to B2, BUTTON3 to B3, BUTTON4 to B4, BUTTON5 to B5, BUTTON6 to B6, BUTTON7 to B7, BUTTON8 to B9, BUTTON9 to B8, LED1 to LED, R10 to R1, R27 to R6, R28 to R5, R29 to R4, R8 to R2, R9 to R3, SCL_SEL to I2C_BUS, SJ_MCP_A0 to A0, SJ_MCP_A1 to A1, SJ_MCP_A2 to A2
Connections:
- net BUTTON0 renamed B0
- net BUTTON1 renamed B1
- net BUTTON2 renamed B2
- net BUTTON3 renamed B3
- removed net BUTTON10: B11.4, U2.GPB2
- removed net BUTTON11: B10.4, U2.GPB3
- removed net BUTTON12: B13.4, U2.GPB4
- removed net BUTTON13: B12.4, U2.GPB5
- removed net BUTTON14: B15.4, U2.GPB6
- removed net BUTTON15: B14.4, U2.GPB7
- removed net BUTTON4: U2.GPA4
- removed net BUTTON5: B4.3, U2.GPA5
- removed net BUTTON6: B5.3, U2.GPA6
- removed net BUTTON7: B6.3, U2.GPA7
- removed net BUTTON8: B7.3, B9.4, U2.GPB0
- removed net BUTTON9: B8.4, U2.GPB1
- new net B10: B10.4, U2.GPB2
- new net B11: B11.4, U2.GPB3
- new net B12: B12.4, U2.GPB4
- new net B13: B13.4, U2.GPB5
- new net B14: B14.4, U2.GPB6
- new net B15: B15.4, U2.GPB7
- new net B4: B4.3, U2.GPA4
- new net B5: B5.3, U2.GPA5
- new net B6: B6.3, U2.GPA6
- new net B7: B7.3, U2.GPA7
- new net B8: B8.4, U2.GPB0
- new net B9: B9.4, U2.GPB1
