File: Chipchestra/chipchestra-v05-analog-inputs.sch (EAGLE design)
At the start: 17 parts

Commit message: updates to chipchestra
Parts:
- renumbered J19 to J9
Changed lines of the file:
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@@
 <?xml version="1.0" encoding="utf-8"?>
 <!DOCTYPE eagle SYSTEM "eagle.dtd">
-<eagle version="8.0.0">
+<eagle version="8.0.1">
 <drawing>
 <settings>
@@
 <part name="FADER7" library="adafruit" deviceset="TRIMPOT" device="3386"/>
 <part name="FADER8" library="adafruit" deviceset="TRIMPOT" device="3386"/>
-<part name="J19" library="SparkFun-Connectors" deviceset="CONN_05X2" device="SHD_LOCK"/>
+<part name="J9" library="SparkFun-Connectors" deviceset="CONN_05X2" device="SHD_LOCK"/>
 <part name="P+3" library="microbuilder" deviceset="VCC" device=""/>
 <part name="SUPPLY3" library="supply2" deviceset="GND" device=""/>
@@
 <instance part="FADER7" gate="G$1" x="96.52" y="2.54" rot="R180"/>
 <instance part="FADER8" gate="G$1" x="96.52" y="-12.7" rot="R180"/>
-<instance part="J19" gate="G$1" x="30.48" y="40.64"/>
+<instance part="J9" gate="G$1" x="30.48" y="40.64"/>
 <instance part="P+3" gate="VCC" x="15.24" y="58.42"/>
 <instance part="SUPPLY3" gate="GND" x="45.72" y="33.02"/>
@@
 </segment>
 <segment>
-<pinref part="J19" gate="G$1" pin="10"/>
+<pinref part="J9" gate="G$1" pin="10"/>
 <wire x1="38.1" y1="35.56" x2="45.72" y2="35.56" width="0.1524" layer="91"/>
 <pinref part="SUPPLY3" gate="GND" pin="GND"/>
@@
 </segment>
 <segment>
-<pinref part="J19" gate="G$1" pin="2"/>
+<pinref part="J9" gate="G$1" pin="2"/>
 <wire x1="38.1" y1="45.72" x2="48.26" y2="45.72" width="0.1524" layer="91"/>
 <label x="48.26" y="45.72" size="1.27" layer="95" xref="yes"/>
@@
 </segment>
 <segment>
-<pinref part="J19" gate="G$1" pin="6"/>
+<pinref part="J9" gate="G$1" pin="6"/>
 <wire x1="38.1" y1="40.64" x2="48.26" y2="40.64" width="0.1524" layer="91"/>
 <label x="48.26" y="40.64" size="1.27" layer="95" xref="yes"/>
@@
 </segment>
 <segment>
-<pinref part="J19" gate="G$1" pin="5"/>
+<pinref part="J9" gate="G$1" pin="5"/>
 <wire x1="22.86" y1="40.64" x2="10.16" y2="40.64" width="0.1524" layer="91"/>
 <label x="10.16" y="40.64" size="1.27" layer="95" rot="R180" xref="yes"/>
@@
 </segment>
 <segment>
-<pinref part="J19" gate="G$1" pin="4"/>
+<pinref part="J9" gate="G$1" pin="4"/>
 <wire x1="38.1" y1="43.18" x2="48.26" y2="43.18" width="0.1524" layer="91"/>
 <label x="48.26" y="43.18" size="1.27" layer="95" xref="yes"/>
@@
 </segment>
 <segment>
-<pinref part="J19" gate="G$1" pin="3"/>
+<pinref part="J9" gate="G$1" pin="3"/>
 <wire x1="22.86" y1="43.18" x2="10.16" y2="43.18" width="0.1524" layer="91"/>
 <label x="10.16" y="43.18" size="1.27" layer="95" rot="R180" xref="yes"/>
@@
 </segment>
 <segment>
-<pinref part="J19" gate="G$1" pin="1"/>
+<pinref part="J9" gate="G$1" pin="1"/>
 <wire x1="22.86" y1="45.72" x2="10.16" y2="45.72" width="0.1524" layer="91"/>
 <label x="10.16" y="45.72" size="1.27" layer="95" rot="R180" xref="yes"/>
@@
 <net name="VCC" class="0">
 <segment>
-<pinref part="J19" gate="G$1" pin="9"/>
+<pinref part="J9" gate="G$1" pin="9"/>
 <wire x1="22.86" y1="35.56" x2="15.24" y2="35.56" width="0.1524" layer="91"/>
 <wire x1="15.24" y1="55.88" x2="15.24" y2="35.56" width="0.1524" layer="91"/>
@@
 </segment>
 <segment>
-<pinref part="J19" gate="G$1" pin="7"/>
+<pinref part="J9" gate="G$1" pin="7"/>
 <wire x1="22.86" y1="38.1" x2="10.16" y2="38.1" width="0.1524" layer="91"/>
 <label x="10.16" y="38.1" size="1.27" layer="95" rot="R180" xref="yes"/>
@@
 </segment>
 <segment>
-<pinref part="J19" gate="G$1" pin="8"/>
+<pinref part="J9" gate="G$1" pin="8"/>
 <wire x1="38.1" y1="38.1" x2="48.26" y2="38.1" width="0.1524" layer="91"/>
 <label x="48.26" y="38.1" size="1.27" layer="95" xref="yes"/>
