File: Mixer-Analog-LM3900/Mixer-Analog-LM3900-Rev-B.sch (EAGLE design)
At the start: 80 parts, among them IC2 LM3900D, IC3 LM3900D, IC5 LM3900D, J1 SJ-3524-SMT, J11 SJ-3524-SMT, J12 SJ-3524-SMT, J2 SJ-3524-SMT, J5 SJ-3524-SMT, J6 SJ-3524-SMT, J7 SJ-3524-SMT

Commit message: new version so of piezo pickups
Parts:
- removed C10, C11, C12, C13, C18, C19, C20, C21, C8, C9: 0.47u, SparkFun-Passives:CAP_POL1206-KIT
- removed IC3, IC5: LM3900D, linear:LM3900D
- removed J11, J12, J2, J5, J6: SJ-3524-SMT, con-cuistack:SJ-3524-SMT
- removed R13, R14, R15, R33, R34, R35, R36, R65, R66, R67, R68: 1M, SparkFun-Passives:RESISTOR1206
- removed R21, R22, R23, R24, R37, R38, R39, R40, R69, R70, R71, R72: 330, SparkFun-Passives:RESISTOR1206
- removed R25, R26, R27, R28, R29, R30, R31, R32, R41, R42, R43, R44, R45, R46, R47, R48, R73, R74, R75, R76, R77, R78, R79, R80: 470, SparkFun-Passives:RESISTOR1206
- removed U$10, U$11, U$3, U$4, U$5, U$6, U$7: POT-DUAL-ALPS-RK10J12E0A0A, CMU-ArtFab:POT-DUAL-ALPS-RK10J12E0A0A
- added C2, C4: 10uF, SparkFun-Passives:CAP_POL1206-KIT
- added R1, R10, R2: 10k, CMU-ArtFab:POT-DUAL-ALPS-RK10J12E0A0A
- added R11, R12: 10k, SparkFun-Passives:RESISTOR1206
- C1, C3: value 0.47u -> 10uF
- renumbered C6 to C1, C7 to C3, IC2 to IC1
Connections:
- removed net N$100: IC5D.OUT, R68.2, R72.2, R80.2
- removed net N$101: C21.-, IC5D.-IN, R68.1, R76.2
- removed net N$102: R72.1, R76.1
- removed net N$103: C21.+, U$10.P$5
- removed net N$104: C20.+, U$10.P$4
- removed net N$105: C19.+, U$11.P$5
- removed net N$106: C18.+, U$11.P$4
- removed net N$107: J11.T, J11.TS, U$11.P$2
- removed net N$108: J12.T, J12.TS, U$10.P$2
- removed net N$109: J12.R, U$10.P$3
- removed net N$110: J11.R, U$11.P$3
- removed net N$112: R30.1, R32.1, R46.1, R48.1, R78.1, R80.1, U$7.P$2
- removed net N$23: R21.1, R25.1
- removed net N$25: C3.-, IC1B.-IN, R14.1, R26.2
- removed net N$26: R22.1, R26.1
- removed net N$27: IC1C.OUT, R15.2, R23.2, R31.2
- removed net N$28: C8.-, IC1C.-IN, R15.1, R27.2
- removed net N$29: R23.1, R27.1
- removed net N$30: IC1D.OUT, R16.2, R24.2, R32.2
- removed net N$31: C9.-, IC1D.-IN, R16.1, R28.2
- removed net N$32: R24.1, R28.1
- removed net N$33: C9.+, U$3.P$5
- removed net N$34: C8.+, U$3.P$4
- removed net N$38: J2.T, J2.TS, U$3.P$2
- removed net N$39: J2.R, U$3.P$3
- removed net N$43: IC3A.OUT, R33.2, R37.2, R45.2
- removed net N$44: C10.-, IC3A.-IN, R33.1, R41.2
- removed net N$45: R37.1, R41.1
- removed net N$46: IC3B.OUT, R34.2, R38.2, R46.2
- removed net N$47: C11.-, IC3B.-IN, R34.1, R42.2
- removed net N$48: R38.1, R42.1
- removed net N$49: IC3C.OUT, R35.2, R39.2, R47.2
- removed net N$50: C12.-, IC3C.-IN, R35.1, R43.2
- removed net N$51: R39.1, R43.1
- removed net N$52: IC3D.OUT, R36.2, R40.2, R48.2
- removed net N$53: C13.-, IC3D.-IN, R36.1, R44.2
- removed net N$54: R40.1, R44.1
- removed net N$55: C13.+, U$5.P$5
- removed net N$56: C12.+, U$5.P$4
- removed net N$57: C11.+, U$6.P$5
- removed net N$58: C10.+, U$6.P$4
- removed net N$59: J5.T, J5.TS, U$6.P$2
- removed net N$60: J6.T, J6.TS, U$5.P$2
- removed net N$64: J6.R, U$5.P$3
- removed net N$66: J5.R, U$6.P$3
- removed net N$91: IC5A.OUT, R65.2, R69.2, R77.2
- removed net N$92: C18.-, IC5A.-IN, R65.1, R73.2
- removed net N$93: R69.1, R73.1
- removed net N$94: IC5B.OUT, R66.2, R70.2, R78.2
- removed net N$95: C19.-, IC5B.-IN, R66.1, R74.2
- removed net N$96: R70.1, R74.1
- removed net N$97: IC5C.OUT, R67.2, R71.2, R79.2
- removed net N$98: C20.-, IC5C.-IN, R67.1, R75.2
- removed net N$99: R71.1, R75.1
- new net N$1: C3.-, IC1B.-IN, R2.P$4
- new net N$2: IC1A.+IN, IC1B.+IN, R11.1, R12.2
- new net N$6: J1.S
- new net N$7: C4.-, R10.P$2
- net 5V: now also R11.2; no longer IC3P.V+, IC5P.V+
- net GND: now also R12.1; no longer IC1A.+IN, IC1B.+IN, IC1C.+IN, IC1D.+IN, IC3A.+IN, IC3B.+IN, IC3C.+IN, IC3D.+IN, IC3P.GND, IC5A.+IN, IC5B.+IN, IC5C.+IN, IC5D.+IN, IC5P.GND, J1.S, J11.S, J12.S, J2.S, J5.S, J6.S
- net N$111: now also C2.-, R10.P$3; no longer R29.1, R31.1, R45.1, R47.1, R77.1, R79.1, U$7.P$3
- net N$18: now also C2.+, R2.P$2; no longer R13.2, R21.2, R29.2
- net N$21: now also R2.P$5; no longer R13.1, R25.2
- net N$24: now also C4.+; no longer R14.2, R22.2, R30.2
- net N$35: now also R1.P$5; no longer U$4.P$5
- net N$36: now also R1.P$4; no longer U$4.P$4
- net N$37: now also R1.P$2; no longer U$4.P$2
- net N$40: now also R1.P$3; no longer U$4.P$3
- net N$61: now also R10.P$4; no longer U$7.P$4
- net N$62: now also R10.P$5; no longer U$7.P$5
Other:
- moved on the sheet: C5, J1, J7, J8, JP1
