File: Mixer-Analog/Mixer-Analog-OPA4134-Rev-K-multi.sch (EAGLE design)
At the start: 114 parts, among them IC1 DMN2400, IC2 BQ21040, IC3 BQ297X, IC4 OPA4134D, IC5 SC4503, IC6 TPS7A49, J1 TRS-1/8"-3.5MM, J10 PHONES-OUT, J11 12V, J2 TRS-1/8"-3.5MM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

Commit message: Add files via upload
Parts:
- R49: value 91.2k -> 100k
- R50: value 100k -> 11k
Changed lines of the file:
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@@
 <?xml version="1.0" encoding="utf-8"?>
 <!DOCTYPE eagle SYSTEM "eagle.dtd">
-<eagle version="8.5.2">
+<eagle version="8.6.0">
 <drawing>
 <settings>
@@
 <part name="P+18" library="supply1" library_urn="urn:adsk.eagle:library:371" deviceset="+12V" device=""/>
 <part name="IC6" library="CMU-ArtFab" deviceset="TPS7A49" device=""/>
-<part name="R49" library="CMU-ArtFab" deviceset="R-US_" device="R0603" value="91.2k"/>
-<part name="R50" library="CMU-ArtFab" deviceset="R-US_" device="R0603" value="100k"/>
+<part name="R49" library="CMU-ArtFab" deviceset="R-US_" device="R0603" value="100k"/>
+<part name="R50" library="CMU-ArtFab" deviceset="R-US_" device="R0603" value="11k"/>
 <part name="GND9" library="SparkFun" deviceset="GND" device=""/>
 <part name="P+16" library="supply1" library_urn="urn:adsk.eagle:library:371" deviceset="V+" device=""/>
